File: PCB/PCB_V0/Tracker/SUN.kicad_sch (KiCad schematic)
At the start: 12 parts

Commit message: Add PCB with GNSS
Parts:
- removed C8 (x2), C9 (x2): 100nF, Capacitor_THT:C_Rect_L7.0mm_W2.0mm_P5.00mm, symbol Device:C
- removed R2 (x2), R3 (x2): LDR03, OptoDevice:R_LDR_10x8.5mm_P7.6mm_Vertical, symbol Sensor_Optical:LDR03
- removed R7 (x2), R8 (x2): 100k, Resistor_THT:R_Axial_DIN0204_L3.6mm_D1.6mm_P5.08mm_Horizontal, symbol Device:R
