File: PCB/PCB_V0/Tracker/Tracker.kicad_pcb (KiCad board)
At the start: 2 copper layers, 49 parts, among them J1 Battery, J2 SPI_Programming, J3 Wind, Q1 BC337, U1 L7805, U2 ATmega328P-P, U3 74HC123, U4 TL082, Y1 16MHz

Commit message: Add PCB with GNSS
Parts:
- removed C10, C11, C7: 1nF, Capacitor_THT:C_Rect_L7.0mm_W2.0mm_P5.00mm
- removed C12, C13, C9: 100nF, Capacitor_THT:C_Rect_L7.0mm_W2.0mm_P5.00mm
- removed D4, D5: 1N4818, Diode_THT:D_DO-41_SOD81_P7.62mm_Horizontal
- removed J2: SPI_Programming, Connector_PinHeader_2.54mm:PinHeader_2x05_P2.54mm_Vertical
- removed Q1: BC337, Package_TO_SOT_THT:TO-92_Inline
- removed R10, R11, R13, R14, R15, R16: 10k, Resistor_THT:R_Axial_DIN0204_L3.6mm_D1.6mm_P5.08mm_Horizontal
- removed R12: 47k, Resistor_THT:R_Axial_DIN0204_L3.6mm_D1.6mm_P5.08mm_Horizontal
- removed R17, R19: 100k, Resistor_THT:R_Axial_DIN0204_L3.6mm_D1.6mm_P5.08mm_Horizontal
- removed R18, R20: LDR03, OptoDevice:R_LDR_10x8.5mm_P7.6mm_Vertical
- removed R5: 270k, Resistor_THT:R_Axial_DIN0204_L3.6mm_D1.6mm_P5.08mm_Horizontal
- removed U4: TL082, Package_DIP:DIP-8_W7.62mm
- added C3: 100nF, Capacitor_THT:C_Rect_L7.0mm_W2.0mm_P5.00mm, F.Cu at (141.8, 97.3)
- added D7: LED, LED_THT:LED_D3.0mm, F.Cu at (160.6, 59.9)
- added H1: MountingHole, MountingHole:MountingHole_3mm, F.Cu at (143.8, 57.0)
- added H2: MountingHole, MountingHole:MountingHole_3mm, F.Cu at (197.8, 56.2)
- added H3: MountingHole, MountingHole:MountingHole_3mm, F.Cu at (198.2, 119.3)
- added H4: MountingHole, MountingHole:MountingHole_3mm, F.Cu at (143.2, 128.3)
- added J10: 132134, Connector_Coaxial:SMA_Molex_73251-1153_EdgeMount_Horizontal, F.Cu at (188.7, 128.3)
- added J11: SPI_Programming, Connector_PinHeader_2.54mm:PinHeader_2x05_P2.54mm_Vertical, F.Cu at (193.3, 85.7)
- added J12: Battery, TerminalBlock_Phoenix:TerminalBlock_Phoenix_MKDS-1,5-2-5.08_1x02_P5.08mm_Horizontal, F.Cu at (17.2, 25.4)
- added J4: RX, Connector_PinHeader_2.54mm:PinHeader_1x01_P2.54mm_Vertical, F.Cu at (172.8, 71.0)
- added J5: TX, Connector_PinHeader_2.54mm:PinHeader_1x01_P2.54mm_Vertical, F.Cu at (172.8, 73.9)
- added J6: GND, Connector_PinHeader_2.54mm:PinHeader_1x01_P2.54mm_Vertical, F.Cu at (149.2, 79.3)
- added J7: GND, Connector_PinHeader_2.54mm:PinHeader_1x01_P2.54mm_Vertical, F.Cu at (149.2, 82.1)
- added J8: GND, Connector_PinHeader_2.54mm:PinHeader_1x01_P2.54mm_Vertical, F.Cu at (149.2, 84.9)
- added J9: Header_LED, Connector_PinHeader_2.54mm:PinHeader_2x01_P2.54mm_Vertical, F.Cu at (168.9, 59.5)
- added U7: GK9501, RF_GPS:ublox_NEO, F.Cu at (182.8, 117.1)
- added U9: L298N, Package_TO_SOT_THT:TO-220-15_P2.54x2.54mm_StaggerOdd_Lead4.58mm_Vertical, F.Cu at (35.3, 37.3)
- C8: value 100nF -> 20F; footprint Capacitor_THT:C_Rect_L7.0mm_W2.0mm_P5.00mm -> Capacitor_THT:C_Radial_D10.0mm_H20.0mm_P5.00mm
- D2: value 1N4818 -> D
- D3: value LED -> D; footprint LED_THT:LED_D5.0mm -> Diode_THT:D_DO-41_SOD81_P7.62mm_Horizontal
- J1, J3: footprint Connector_Molex:Molex_KK-396_A-41791-0002_1x02_P3.96mm_Vertical -> TerminalBlock_Phoenix:TerminalBlock_Phoenix_MKDS-1,5-2-5.08_1x02_P5.08mm_Horizontal
- R2: value 100k -> 1k
- R3: value LDR03 -> 1k; footprint OptoDevice:R_LDR_10x8.5mm_P7.6mm_Vertical -> Resistor_THT:R_Axial_DIN0204_L3.6mm_D1.6mm_P5.08mm_Horizontal
- R6: value 100k -> 220
- R7: value 100k -> 270
- R8: value LDR03 -> 330; footprint OptoDevice:R_LDR_10x8.5mm_P7.6mm_Vertical -> Resistor_THT:R_Axial_DIN0204_L3.6mm_D1.6mm_P5.08mm_Horizontal
- R9: value 10k -> 100
- U3: value 74HC123 -> LM317_TO-220; footprint Package_DIP:DIP-16_W7.62mm -> Package_TO_SOT_THT:TO-220-3_Vertical
- moved C8 91.0 mm to (150.9, 109.3), turned to 180 degrees
- moved J3 86.7 mm to (182.0, 60.3), turned to 180 degrees
- moved R8 83.0 mm to (149.7, 102.5)
- moved R3 81.3 mm to (172.4, 108.0), turned to 0 degrees
- moved R4 76.6 mm to (172.3, 59.5)
- moved R2 67.6 mm to (179.5, 108.0), turned to 0 degrees
- moved D3 54.4 mm to (153.6, 103.2)
- moved R7 49.6 mm to (161.1, 63.3)
- moved R6 41.6 mm to (144.8, 95.3)
- moved U3 28.5 mm to (149.3, 98.1), turned to 90 degrees
- moved R9 27.1 mm to (159.8, 111.4), turned to 180 degrees
- moved D2 14.0 mm to (156.9, 103.2), turned to 90 degrees
Connections:
- net Net-(D1-K) renamed +BATT
- C8 pad 1: GND -> Net-(C8-Pad1)
- C8 pad 2: /SUN/LDR1 -> GND
- D2 pad 1: Net-(D2-K) -> +3.3V
- D2 pad 2: GND -> +3V8
- D3 pad 1: GND -> /GNSS/Vcapa
- D3 pad 2: Net-(D3-A) -> +3V8
- J3 pad 1: Net-(J3-Pin_1) -> /WIND/OUT
- R2 pad 1: +5V -> /GNSS/RX
- R2 pad 2: /SUN/LDR1 -> GND
- R3 pad 1: /SUN/LDR1 -> +3.3V
- R3 pad 2: GND -> /GNSS/RX
- R4 pad 2: Net-(J3-Pin_1) -> /WIND/OUT
- R6 pad 1: +5V -> +3V8
- R6 pad 2: Net-(U3A-Cext) -> Net-(U3-ADJ)
- R7 pad 1: +5V -> Net-(D7-K)
- R7 pad 2: /SUN/LDR2 -> GND
- R8 pad 1: /SUN/LDR2 -> Net-(U3-ADJ)
- R9 pad 1: Net-(U3A-Q) -> /GNSS/Vcapa
- R9 pad 2: Net-(C11-Pad2) -> Net-(C8-Pad1)
- U2 pad 14: unconnected-(U2-PB0-Pad14) -> /GNSS/RX
- U2 pad 15: unconnected-(U2-PB1-Pad15) -> /GNSS/TX
- U2 pad 16: unconnected-(U2-PB2-Pad16) -> /GNSS/PPS
- U2 pad 2: unconnected-(U2-PD0-Pad2) -> Net-(J4-Pin_1)
- U2 pad 23: /SUN/LDR1 -> unconnected-(U2-PC0-Pad23)
- U2 pad 24: /SUN/LDR2 -> unconnected-(U2-PC1-Pad24)
- U2 pad 25: /SUN/LDR3 -> unconnected-(U2-PC2-Pad25)
- U2 pad 26: /SUN/LDR4 -> unconnected-(U2-PC3-Pad26)
- U2 pad 27: /SDA -> unconnected-(U2-PC4-Pad27)
- U2 pad 28: /SCL -> unconnected-(U2-PC5-Pad28)
- U2 pad 3: unconnected-(U2-PD1-Pad3) -> Net-(J5-Pin_1)
- U2 pad 5: /WIND/SECURITY -> unconnected-(U2-PD3-Pad5)
- U3 pad 1: Net-(D2-K) -> Net-(U3-ADJ)
- U3 pad 2: unconnected-(U3A-B-Pad2) -> +3V8
- U3 pad 3: unconnected-(U3A-Clr-Pad3) -> +5V
Routing:
- net Net-(J12-Pin_1): track 0.00 -> 49.2 mm
- net +3.3V: track 0.00 -> 40.1 mm
- net /MOSI: track 0.00 -> 37.3 mm
- net Net-(J12-Pin_2): track 0.00 -> 31.4 mm
- net /WIND/OUT: track 0.00 -> 26.3 mm
- net /SUN/LDR1: track 23.8 -> 0.00 mm
- net +3V8: track 0.00 -> 16.1 mm
- net /RST: track 7.23 -> 20.2 mm, vias 0 -> 1
- net Net-(D2-K): track 12.5 -> 0.00 mm
- net /GNSS/Vcapa: track 0.00 -> 11.4 mm
- net +5V: track 37.0 -> 47.8 mm
- net /GNSS/RX: track 0.00 -> 10.5 mm
- net Net-(U3-ADJ): track 0.00 -> 9.97 mm
- net /GNSS/TX: track 0.00 -> 9.00 mm
- net Net-(J10-In): track 0.00 -> 6.90 mm
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Other:
- board outline added: 63.8 x 80.7 mm
