File: Hardware/Tracker.kicad_pcb (KiCad board)
At the start: 2 copper layers, 99 parts, among them J1 Battery, J10 132134, J11 SPI_Programming, J12 Sortie Moteur, J13 Position_Potentiometer, J15 Screw_Terminal_01x04, J2 +24V, J3 Wind, J4 RX, J5 TX, J6 GND, J7 GND, J8 GND, J9 Haeder_LED, Q1 IRF4905, Q2 IRF520, Q3 2N7000, Q4 IRF4905, Q5 IRF520, Q6 IRF4905, Q7 2N7000, SW1 SW_Push, U1 L7805, U10 PC817, U11 PC817, U12 PC817, U2 ATmega328P-P, U3 LM317_TO-220, U4 PC817, U5 74HC123, U6 LM358, U7 GK9501, U8 PC817, Y1 16MHz

Commit message: Update
Parts:
- removed C10, C11, C7, C9: 100nF, Capacitor_THT:C_Rect_L7.0mm_W2.0mm_P5.00mm
- removed D12: 3.3V, Diode_THT:D_A-405_P10.16mm_Horizontal
- removed J12: Sortie Moteur, TerminalBlock_Phoenix:TerminalBlock_Phoenix_MKDS-3-2-5.08_1x02_P5.08mm_Horizontal
- removed J13: Position_Potentiometer, TerminalBlock_Phoenix:TerminalBlock_Phoenix_MKDS-1,5-3-5.08_1x03_P5.08mm_Horizontal
- removed J15: Screw_Terminal_01x04, TerminalBlock_Phoenix:TerminalBlock_Phoenix_MPT-0,5-4-2.54_1x04_P2.54mm_Horizontal
- removed the J2 at (136.8, 36.9)
- removed the J3 at (116.5, 134.7)
- removed the R12 at (150.7, 128.6)
- removed R27, R29: 470, Resistor_THT:R_Axial_DIN0207_L6.3mm_D2.5mm_P7.62mm_Horizontal
- removed R28, R31, R35: 1K, Resistor_THT:R_Axial_DIN0207_L6.3mm_D2.5mm_P7.62mm_Horizontal
- removed R30, R37: 2.2K, Resistor_THT:R_Axial_DIN0207_L6.3mm_D2.5mm_P7.62mm_Horizontal
- removed R32: 100k, Resistor_THT:R_Axial_DIN0207_L6.3mm_D2.5mm_P7.62mm_Horizontal
- removed R33: 1k, Resistor_THT:R_Axial_DIN0207_L6.3mm_D2.5mm_P7.62mm_Horizontal
- removed R34: 2.7K, Resistor_THT:R_Axial_DIN0207_L6.3mm_D2.5mm_P7.62mm_Horizontal
- removed R38: 3.3K, Resistor_THT:R_Axial_DIN0207_L6.3mm_D2.5mm_P7.62mm_Horizontal
- removed the R4 at (132.2, 125.8)
- removed the R5 at (135.5, 127.3)
- removed U10, U11, U12, U8: PC817, Package_DIP:DIP-4_W7.62mm
- removed U6: LM358, Package_DIP:DIP-8_W7.62mm_Socket
- added C1: 100n, Capacitor_SMD:C_0603_1608Metric, F.Cu at (149.1, 120.1)
- added C2: 1n, Capacitor_SMD:C_0603_1608Metric, F.Cu at (133.3, 107.4)
- added C3: 100n, Capacitor_THT:C_Radial_D4.0mm_H5.0mm_P1.50mm, F.Cu at (147.8, 106.4)
- added D1: LED, LED_THT:LED_D3.0mm, F.Cu at (180.8, 34.8)
- added D1: LED, LED_THT:LED_D5.0mm, F.Cu at (110.7, 109.5)
- added D10: 1N4148, Diode_THT:D_DO-35_SOD27_P7.62mm_Horizontal, F.Cu at (132.1, 80.0)
- added D14: 1N5408, Diode_THT:D_DO-201AD_P15.24mm_Horizontal, F.Cu at (140.9, 34.3)
- added D2: LED, LED_THT:LED_D3.0mm, F.Cu at (180.9, 43.0)
- added D3: D_Dual_CommonCathode_AAK, Package_TO_SOT_THT:TO-220-3_Vertical, F.Cu at (165.5, 56.0)
- added D6: LED, LED_THT:LED_D3.0mm, F.Cu at (134.9, 84.3)
- added D7: LED, LED_THT:LED_D3.0mm, F.Cu at (200.7, 84.6)
- added F1: Fuse, Fuse:Fuseholder_Cylinder-5x20mm_Schurter_0031_8201_Horizontal_Open, F.Cu at (148.4, 37.5)
- added H1: MountingHole, MountingHole:MountingHole_3mm, F.Cu at (143.0, 100.8)
- added H1: Probe_GND, Holes:Hole_1mm_Scope, F.Cu at (148.1, 93.2)
- added H2: Probe_GND, Holes:Hole_1mm_Scope, F.Cu at (160.8, 49.8)
- added H3: MountingHole, MountingHole:MountingHole_3mm, F.Cu at (218.4, 117.1)
- added H4: MountingHole, MountingHole:MountingHole_3mm, F.Cu at (66.5, 30.2)
- added H5: MountingHole, MountingHole:MountingHole_3mm, F.Cu at (217.9, 30.7)
- added H6: MountingHole, MountingHole:MountingHole_3mm, F.Cu at (106.2, 91.2)
- added H7: Probe_GND, Holes:Hole_1mm_Scope, F.Cu at (117.3, 82.8)
- added H8: Probe_GND, Holes:Hole_1mm_Scope, F.Cu at (214.9, 77.5)
- added J1: output, TerminalBlock_TE-Connectivity:TerminalBlock_TE_282834-2_1x02_P2.54mm_Horizontal, F.Cu at (108.0, 105.2)
- added J1: +24V, TerminalBlock_Phoenix:TerminalBlock_Phoenix_MKDS-1,5-2-5.08_1x02_P5.08mm_Horizontal, F.Cu at (117.5, 35.9)
- added J2: PinHeader_Control, Connector_PinHeader_2.54mm:PinHeader_1x04_P2.54mm_Vertical, F.Cu at (121.7, 51.5)
- added J2: Probe_sensor, Connector_PinHeader_2.54mm:PinHeader_1x01_P2.54mm_Vertical, F.Cu at (159.8, 107.7)
- added J3: Motor, TerminalBlock_Phoenix:TerminalBlock_Phoenix_MKDS-3-2-5.08_1x02_P5.08mm_Horizontal, F.Cu at (165.7, 66.8)
- added J3: Pull_up_strap, Connector_PinHeader_2.54mm:PinHeader_1x02_P2.54mm_Vertical, F.Cu at (160.0, 117.6)
- added J4: LP_Probe, Connector_PinHeader_2.54mm:PinHeader_1x01_P2.54mm_Vertical, F.Cu at (136.7, 104.4)
- added J4: Control, TerminalBlock_Phoenix:TerminalBlock_Phoenix_MPT-0,5-4-2.54_1x04_P2.54mm_Horizontal, F.Cu at (115.9, 59.2)
- added J5: GND, Connector_PinHeader_2.54mm:PinHeader_1x02_P2.54mm_Vertical, F.Cu at (167.6, 101.1)
- added J7: +5V, TerminalBlock_TE-Connectivity:TerminalBlock_TE_282834-2_1x02_P2.54mm_Horizontal, F.Cu at (166.1, 114.8)
- added J8: Sensor, TerminalBlock_TE-Connectivity:TerminalBlock_TE_282834-2_1x02_P2.54mm_Horizontal, F.Cu at (166.1, 107.4)
- added R1: 470k, Resistor_SMD:R_0603_1608Metric, F.Cu at (152.4, 120.1)
- added R1: 1k, Resistor_THT:R_Axial_DIN0207_L6.3mm_D2.5mm_P7.62mm_Horizontal, F.Cu at (164.5, 50.2)
- added R12: 1K, Resistor_THT:R_Axial_DIN0207_L6.3mm_D2.5mm_P7.62mm_Horizontal, F.Cu at (146.1, 61.9)
- added R12: 10k, Resistor_THT:R_Axial_DIN0207_L6.3mm_D2.5mm_P7.62mm_Horizontal, F.Cu at (156.5, 110.7)
- added R16: 100k, Resistor_THT:R_Axial_DIN0207_L6.3mm_D2.5mm_P7.62mm_Horizontal, F.Cu at (145.3, 73.6)
- added R2: 1k, Resistor_SMD:R_0603_1608Metric, F.Cu at (132.1, 112.6)
- added R2: 3.3K, Resistor_THT:R_Axial_DIN0207_L6.3mm_D2.5mm_P7.62mm_Horizontal, F.Cu at (183.6, 34.7)
- added R21: 470, Resistor_THT:R_Axial_DIN0207_L6.3mm_D2.5mm_P7.62mm_Horizontal, F.Cu at (198.1, 85.3)
- added R22: 3.3K, Resistor_THT:R_Axial_DIN0207_L6.3mm_D2.5mm_P7.62mm_Horizontal, F.Cu at (165.1, 87.0)
- added R23: 3.3K, Resistor_THT:R_Axial_DIN0207_L6.3mm_D2.5mm_P7.62mm_Horizontal, F.Cu at (171.7, 87.1)
- added R25: 2.7k, Resistor_THT:R_Axial_DIN0207_L6.3mm_D2.5mm_P7.62mm_Horizontal, F.Cu at (144.6, 33.7)
- added R3: 3.3K, Resistor_THT:R_Axial_DIN0207_L6.3mm_D2.5mm_P7.62mm_Horizontal, F.Cu at (183.9, 42.4)
- added R3: 1k, Resistor_THT:R_Axial_DIN0207_L6.3mm_D2.5mm_P7.62mm_Horizontal, F.Cu at (116.1, 112.5)
- added R4: 1k, Resistor_THT:R_Axial_DIN0207_L6.3mm_D2.5mm_P7.62mm_Horizontal, F.Cu at (129.8, 109.7)
- added R4: 470, Resistor_THT:R_Axial_DIN0207_L6.3mm_D2.5mm_P7.62mm_Horizontal, F.Cu at (130.8, 47.5)
- added R5: 470, Resistor_THT:R_Axial_DIN0207_L6.3mm_D2.5mm_P7.62mm_Horizontal, F.Cu at (116.1, 115.8)
- added R5: 2.2K, Resistor_THT:R_Axial_DIN0207_L6.3mm_D2.5mm_P7.62mm_Horizontal, F.Cu at (153.7, 45.1)
- added R6: 1K, Resistor_THT:R_Axial_DIN0207_L6.3mm_D2.5mm_P7.62mm_Horizontal, F.Cu at (146.0, 58.6)
- added R7: 1K, Resistor_THT:R_Axial_DIN0207_L6.3mm_D2.5mm_P7.62mm_Horizontal, F.Cu at (198.5, 59.6)
- added R8: 470, Resistor_THT:R_Axial_DIN0207_L6.3mm_D2.5mm_P7.62mm_Horizontal, F.Cu at (135.2, 65.8)
- added R9: 2.2K, Resistor_THT:R_Axial_DIN0207_L6.3mm_D2.5mm_P7.62mm_Horizontal, F.Cu at (138.3, 52.6)
- added SW1: SW_B, Button_Switch_THT:SW_PUSH_6mm_H8mm, F.Cu at (131.3, 68.8)
- added SW2: SW_A, Button_Switch_THT:SW_PUSH_6mm_H8mm, F.Cu at (211.8, 68.0)
- added SW3: SW_E, Button_Switch_THT:SW_PUSH_6mm_H8mm, F.Cu at (140.2, 43.3)
- added U1: PC817, Package_DIP:DIP-4_W7.62mm, F.Cu at (143.3, 44.2)
- added U1: 74HC123, Package_DIP:DIP-16_W7.62mm, F.Cu at (152.9, 110.0)
- added U2: PC817, Package_DIP:DIP-4_W7.62mm, F.Cu at (128.1, 52.5)
- added U2: LM358, Package_DIP:DIP-8_W7.62mm, F.Cu at (118.6, 109.7)
- added U3: PC817, Package_DIP:DIP-4_W7.62mm, F.Cu at (198.5, 51.4)
- C4: value 100nF -> 100n; footprint Capacitor_THT:C_Rect_L7.0mm_W2.0mm_P5.00mm -> Capacitor_THT:C_Radial_D4.0mm_H5.0mm_P1.50mm
- D11: value 1N5406 -> 1N4148; footprint Diode_THT:D_DO-201AD_P15.24mm_Horizontal -> Diode_THT:D_DO-35_SOD27_P7.62mm_Horizontal
- D13: value LED -> 1N4148; footprint LED_THT:LED_D3.0mm -> Diode_THT:D_DO-35_SOD27_P7.62mm_Horizontal
- D4, D5: value 1N5406 -> 1N5408
- D8: value 1N5406 -> LED; footprint Diode_THT:D_DO-201AD_P15.24mm_Horizontal -> LED_THT:LED_D3.0mm
- Q2: value IRF520 -> IRF4905
- Q3: value 2N7000 -> IRF4905; footprint Package_TO_SOT_THT:TO-92_Inline -> Package_TO_SOT_THT:TO-220-3_Vertical
- Q4: value IRF4905 -> IRF520
- Q6: value IRF4905 -> 2N7000; footprint Package_TO_SOT_THT:TO-220-3_Vertical -> Package_TO_SOT_THT:TO-92_Inline
- R10: value 10k -> 2.2K
- R11, R15: value 10k -> 470
- R13: value 470 -> 1K
- R14: value 100k -> 470
- R17: value 2.2K -> 100k
- R18: value 1K -> 100k
- R20: value 1K -> 470
- R24: value 470 -> 2.7k
- R26: value 3.3K -> 2.7k
- RV1: value R_Potentiometer -> V_Selector; footprint Potentiometer_THT:Potentiometer_Bourns_3266Y_Vertical -> Potentiometer_THT:Potentiometer_Bourns_3386C_Horizontal
- U5: value 74HC123 -> PC817; footprint Package_DIP:DIP-16_W7.62mm_Socket -> Package_DIP:DIP-4_W7.62mm
- moved C3 168.4 mm to (198.1, 104.1)
- moved C8 168.4 mm to (207.2, 116.1)
- moved D2 168.4 mm to (213.2, 110.0)
- moved D3 168.4 mm to (209.9, 110.1)
- moved R6 168.4 mm to (201.0, 102.1)
- moved R8 168.4 mm to (205.9, 109.3)
- moved U3 168.4 mm to (205.6, 105.0)
- moved SW1 129.2 mm to (78.1, 33.9)
- moved U7 112.4 mm to (184.4, 105.2)
- moved R11 111.6 mm to (202.0, 51.6), turned to -90 degrees
- moved J10 106.0 mm to (183.8, 118.6)
- moved R10 104.3 mm to (198.5, 56.4), turned to 180 degrees
- moved R24 102.7 mm to (205.0, 59.7), turned to 0 degrees
- moved U5 100.4 mm to (207.6, 75.9), turned to 180 degrees
- moved R13 94.5 mm to (197.7, 62.9), turned to -90 degrees
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Connections:
- C4 pad 1: Net-(U5A-RCext) -> /+VCC_Wind
- C4 pad 2: Net-(U5A-Cext) -> GND
- D11 pad 1: +VCC_Motor -> /IN_B
- D13 pad 1: Net-(D13-K) -> /ENABLE
- D13 pad 2: +24V -> Net-(D13-A)
- D4 pad 2: GND_MOTOR -> GND
- D5 pad 1: +VCC_Motor -> Net-(D5-K)
- D5 pad 2: Net-(D4-K) -> GND
- D8 pad 1: Net-(D11-A) -> Net-(D8-K)
- D8 pad 2: GND_MOTOR -> Net-(D4-K)
- D9 pad 2: +VCC_Motor -> Net-(D5-K)
- Q1 pad 2: Net-(D4-K) -> +VCC_Motor
- Q1 pad 3: +VCC_Motor -> Net-(D1-A)
- Q2 pad 3: GND_MOTOR -> +VCC_Motor
- Q3 pad 1: GND_MOTOR -> Net-(Q3-G)
- Q3 pad 2: /Motors/IN_B -> Net-(D5-K)
- Q3 pad 3: Net-(Q3-D) -> +VCC_Motor
- Q4 pad 2: Net-(D11-A) -> Net-(D4-K)
- Q4 pad 3: +VCC_Motor -> GND
- Q5 pad 1: Net-(Q3-D) -> Net-(Q5-G)
- Q5 pad 2: Net-(D11-A) -> Net-(D5-K)
- Q5 pad 3: GND_MOTOR -> GND
- Q6 pad 1: Net-(Q6-G) -> GND
- Q6 pad 2: +VCC_Motor -> /IN_A
- Q6 pad 3: +24V -> Net-(Q4-G)
- Q7 pad 1: GND_MOTOR -> GND
- Q7 pad 2: /Motors/IN_A -> /IN_B
- Q7 pad 3: Net-(Q2-G) -> Net-(Q5-G)
- R10 pad 1: Net-(U5A-Q) -> Net-(R10-Pad1)
- R10 pad 2: Net-(C7-Pad1) -> Net-(Q3-G)
- R11 pad 1: Net-(C7-Pad1) -> Net-(R11-Pad1)
- R11 pad 2: Net-(U6A-+) -> /IN_B
- R13 pad 1: /Motors/IN_A -> +VCC_Motor
- R14 pad 1: /Motors/IN_A -> /IN_B
- R14 pad 2: GND_MOTOR -> Net-(R14-Pad2)
- R15 pad 1: GND_WIND -> Net-(R15-Pad1)
- R15 pad 2: /WIND/Wind_interrupt -> /IN_A
- R17 pad 1: Net-(R17-Pad1) -> Net-(Q5-G)
- R17 pad 2: Net-(Q1-G) -> GND
- R18 pad 1: +VCC_Motor -> /IN_A
- R18 pad 2: Net-(R18-Pad2) -> GND
- R19 pad 1: Net-(Q2-G) -> /IN_B
- R19 pad 2: GND_MOTOR -> GND
- R20 pad 1: +VCC_Motor -> Net-(D6-K)
- R20 pad 2: Net-(Q1-G) -> GND
- R24 pad 1: /Motors/IN_B -> +VCC_Motor
- R26 pad 1: Net-(D9-K) -> +VCC_Motor
- R26 pad 2: GND_MOTOR -> Net-(SW1A-B)
- RV1 pad 1: +5V -> /+VCC_Wind
- RV1 pad 3: GND_WIND -> GND
- U4 pad 1: Net-(R13-Pad2) -> Net-(R14-Pad2)
- U4 pad 2: GND_MOTOR -> GND
- U4 pad 3: GND_MOTOR -> Net-(Q4-G)
- U4 pad 4: Net-(R17-Pad1) -> Net-(R12-Pad2)
- U5 pad 1: unconnected-(U5A-A-Pad1) -> Net-(R15-Pad1)
- U5 pad 2: /WIND/RAW_DATA -> GND
- U5 pad 3: GND_WIND -> Net-(Q5-G)
- U5 pad 4: unconnected-(U5A-~{Q}-Pad4) -> Net-(R13-Pad2)
Routing:
- net /IN_A: track 0.00 -> 163.5 mm
- net /IN_B: track 0.00 -> 138.2 mm
- net /+VCC_Wind: track 0.00 -> 112.2 mm, vias 0 -> 1
- net +VCC_Motor: track 62.7 -> 140.3 mm
- net Net-(D5-K): track 0.00 -> 63.9 mm
- net Net-(D11-A): track 80.1 -> 20.0 mm
- net Net-(D10-A): track 0.00 -> 47.1 mm
- net +24V: track 43.7 -> 8.78 mm
- net /Motors/IN_A: track 35.9 -> 1.51 mm
- net Net-(D1-A): track 7.91 -> 34.6 mm
- net Net-(Q5-G): track 0.00 -> 24.5 mm
- net +5V: track 68.6 -> 47.6 mm
- net GND_MOTOR: track 22.7 -> 3.24 mm
- net +3.3V: track 40.1 -> 20.9 mm
- net Net-(J2-Pin_1): track 0.00 -> 19.1 mm
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- added copper zone on B.Cu, net GND
- added copper zone on F.Cu, net GND
- removed copper zone on B.Cu, net GND_MOTOR
- removed copper zone on F.Cu, net GND_MOTOR
- removed copper zone on B.Cu, net GND_WIND
- removed copper zone on F.Cu, net GND_WIND
Other:
- board outline added: 167.4 x 98.3 mm
- board text added: "+24V"
- board text added: "+24V_ENABLED"
- board text added: "+24V_ON"
- board text added: "CFT - V1"
- board text added: "ENABLE"
- board text added: "GND"
- board text added: "IN_A"
- board text added: "IN_B"
- board text added: "ON_A"
- board text added: "ON_B"
- board text added: "SW_ENABLE"
- board text added: "SW_ON_A"
- board text added: "SW_ON_B"
- board text added: "Tracker solaire - CREPP Carte de contrôle moteur V1.0"

Commit message: Update of PCB
Parts:
- removed the C1 at (84.1, 117.4)
- removed the C1 at (149.1, 120.1)
- removed the C2 at (89.1, 103.7)
- removed the C2 at (133.3, 107.4)
- removed the C3 at (147.8, 106.4)
- removed the C3 at (198.1, 104.1)
- removed the D1 at (180.8, 34.8)
- removed the D1 at (84.0, 114.5)
- removed the D1 at (110.7, 109.5)
- removed the D2 at (213.2, 110.0)
- removed the D2 at (180.9, 43.0)
- removed the D3 at (165.5, 56.0)
- removed the D3 at (209.9, 110.1)
- removed the D7 at (200.7, 84.6)
- removed the D7 at (83.6, 99.2)
- removed F1: Fuse, Fuse:Fuseholder_Cylinder-5x20mm_Schurter_0031_8201_Horizontal_Open
- removed the H1 at (10.9, 54.1)
- removed the H1 at (143.0, 100.8)
- removed the H1 at (148.1, 93.2)
- removed the H2 at (160.8, 49.8)
- removed the H2 at (93.7, 30.2)
- removed the H3 at (67.3, 90.7)
- removed the H3 at (218.4, 117.1)
- removed the H4 at (66.5, 30.2)
- removed the H4 at (9.91, 146.1)
- removed H5, H6: MountingHole, MountingHole:MountingHole_3mm
- removed H7: Probe_GND, Holes:Hole_1mm_Scope
- removed the J1 at (108.0, 105.2)
- removed the J1 at (117.5, 35.9)
- removed the J1 at (76.1, 107.1)
- removed the J2 at (121.7, 51.5)
- removed the J2 at (159.8, 107.7)
- removed the J3 at (165.7, 66.8)
- removed the J3 at (160.0, 117.6)
- removed the J4 at (136.7, 104.4)
- removed the J4 at (115.9, 59.2)
- removed the J4 at (75.0, 45.8)
- removed the J5 at (75.0, 48.7)
- removed the J5 at (167.6, 101.1)
- removed the J7 at (166.1, 114.8)
- removed the J7 at (61.2, 53.1)
- removed the J8 at (166.1, 107.4)
- removed the J8 at (64.8, 53.3)
- removed the R1 at (152.4, 120.1)
- removed the R1 at (164.5, 50.2)
- removed the R1 at (75.4, 51.4)
- removed the R12 at (146.1, 61.9)
- removed the R12 at (156.5, 110.7)
- removed the R16 at (145.3, 73.6)
- removed the R16 at (67.5, 78.8)
- removed the R2 at (132.1, 112.6)
- removed the R2 at (183.6, 34.7)
- removed the R2 at (81.7, 82.8)
- removed the R21 at (198.1, 85.3)
- removed the R21 at (75.4, 75.5)
- removed the R3 at (74.6, 82.8)
- removed the R3 at (183.9, 42.4)
- removed the R3 at (116.1, 112.5)
- removed the R4 at (129.8, 109.7)
- removed the R4 at (130.8, 47.5)
- removed the R5 at (116.1, 115.8)
- removed the R5 at (153.7, 45.1)
- removed the R6 at (201.0, 102.1)
- removed the R6 at (146.0, 58.6)
- removed the R7 at (198.5, 59.6)
- removed the R7 at (84.1, 102.6)
- removed the R8 at (135.2, 65.8)
- removed the R8 at (205.9, 109.3)
- removed the R9 at (138.3, 52.6)
- removed the R9 at (195.6, 113.5)
- removed the SW1 at (78.1, 33.9)
- removed the SW1 at (131.3, 68.8)
- removed the U1 at (143.3, 44.2)
- removed the U1 at (152.9, 110.0)
- removed the U1 at (89.4, 114.5)
- removed the U2 at (78.0, 45.3)
- removed the U2 at (128.1, 52.5)
- removed the U2 at (118.6, 109.7)
- removed the U3 at (198.5, 51.4)
- removed the U3 at (205.6, 105.0)
- added AE1: Internal_antenna, MountingHole:MountingHole_2.2mm_M2_DIN965_Pad, F.Cu at (132.4, 146.3)
- added C1: 100nF, Capacitor_THT:C_Radial_D5.0mm_H11.0mm_P2.00mm, F.Cu at (72.8, 105.9)
- added C10: 1mF, Capacitor_THT:C_Radial_D10.0mm_H16.0mm_P5.00mm, F.Cu at (63.5, 41.4)
- added C11: 100nF, Capacitor_THT:C_Radial_D5.0mm_H11.0mm_P2.00mm, F.Cu at (66.7, 57.0)
- added C12: 100nF, Capacitor_THT:C_Radial_D5.0mm_H11.0mm_P2.00mm, F.Cu at (79.4, 51.2)
- added C13: 100nF, Capacitor_THT:C_Radial_D5.0mm_H11.0mm_P2.00mm, F.Cu at (92.7, 61.2)
- added C14: 100nF, Capacitor_THT:C_Radial_D5.0mm_H11.0mm_P2.00mm, F.Cu at (64.3, 62.4)
- added C15: 20F, Capacitor_THT:C_Radial_D10.0mm_H20.0mm_P5.00mm, F.Cu at (64.8, 70.9)
- added C16: 100nF, Capacitor_SMD:C_0603_1608Metric, B.Cu at (132.3, 131.0)
- added C17: 100nF, Capacitor_THT:C_Radial_D5.0mm_H11.0mm_P2.00mm, F.Cu at (77.8, 77.7)
- added C18: 100nF, Capacitor_SMD:C_0603_1608Metric, B.Cu at (141.9, 131.1)
- added C19: 100nF, Capacitor_THT:C_Radial_D5.0mm_H11.0mm_P2.00mm, F.Cu at (63.6, 115.0)
- added C2: 100nF, Capacitor_THT:C_Radial_D5.0mm_H11.0mm_P2.00mm, F.Cu at (158.3, 103.1)
- added C20: 100pF, Capacitor_SMD:C_0603_1608Metric, B.Cu at (113.5, 149.8)
- added C22: 100pF, Capacitor_SMD:C_0603_1608Metric, B.Cu at (129.0, 140.9)
- added C23: 100pF, Capacitor_SMD:C_0603_1608Metric, B.Cu at (128.2, 132.8)
- added C3: 100nF, Capacitor_SMD:C_0603_1608Metric, F.Cu at (153.9, 108.5)
- added C7: 22pF, Capacitor_THT:C_Disc_D4.7mm_W2.5mm_P5.00mm, F.Cu at (100.5, 94.8)
- added C9: 100nF, Capacitor_THT:C_Radial_D5.0mm_H11.0mm_P2.00mm, F.Cu at (68.2, 38.1)
- added D1: LED, LED_THT:LED_D3.0mm, F.Cu at (168.8, 35.1)
- added D12: LED, LED_THT:LED_D3.0mm, F.Cu at (90.2, 66.2)
- added D15: LED, LED_THT:LED_D3.0mm, F.Cu at (63.2, 49.6)
- added D16: LED, LED_THT:LED_D3.0mm, F.Cu at (75.3, 58.6)
- added D17: 1N4818, Diode_THT:D_DO-41_SOD81_P7.62mm_Horizontal, F.Cu at (47.3, 65.2)
- added D18: LED, LED_THT:LED_D3.0mm, F.Cu at (187.4, 131.8)
- added D19: LED, LED_SMD:LED_0603_1608Metric, B.Cu at (140.5, 138.6)
- added D2: LED, LED_THT:LED_D3.0mm, F.Cu at (168.9, 43.3)
- added D24: 1N4818, Diode_THT:D_DO-41_SOD81_P7.62mm_Horizontal, F.Cu at (70.9, 32.3)
- added D3: D_Dual_CommonCathode_AAK, Package_TO_SOT_THT:TO-220-3_Vertical, F.Cu at (153.5, 56.3)
- added D7: LED, LED_THT:LED_D3.0mm, F.Cu at (188.6, 84.9)
- added H1: MountingHole, MountingHole:MountingHole_3mm, F.Cu at (30.1, 148.6)
- added H10: MountingHole_Pad, MountingHole:MountingHole_3.2mm_M3_Pad, F.Cu at (151.4, 32.6)
- added H2: MountingHole, MountingHole:MountingHole_3mm, F.Cu at (51.6, 38.5)
- added H3: MountingHole, MountingHole:MountingHole_3mm, F.Cu at (197.3, 46.1)
- added H4: MountingHole, MountingHole:MountingHole_3mm, F.Cu at (197.4, 129.4)
- added H9: MountingHole_Pad, MountingHole:MountingHole_3.2mm_M3_Pad, F.Cu at (139.3, 32.7)
- added HS5: Heatsink, HeatSink:HeastSink_MOSFET_15mm_10mm_20mm, F.Cu at (156.3, 46.9)
- added J1: +24V, TerminalBlock_Phoenix:TerminalBlock_Phoenix_MKDS-1,5-2-5.08_1x02_P5.08mm_Horizontal, F.Cu at (108.5, 32.6)
- added J100: 132134, Connector_Coaxial:SMA_Molex_73251-1153_EdgeMount_Horizontal, F.Cu at (113.5, 155.6)
- added J12: Conn_02x06_Odd_Even, Connector_PinHeader_2.54mm:PinHeader_2x06_P2.54mm_Vertical, F.Cu at (89.7, 123.8)
- added J13: RAW_data_Wind, Connector_PinHeader_2.54mm:PinHeader_1x01_P2.54mm_Vertical, F.Cu at (239.3, 106.7)
- added J14: OLED_SOCKET, Connector_PinSocket_2.54mm:PinSocket_1x04_P2.54mm_Vertical, F.Cu at (77.6, 130.6)
- added J15: SPI_Programming, Connector_PinHeader_2.54mm:PinHeader_2x05_P2.54mm_Vertical, F.Cu at (56.9, 102.3)
- added J16: I2C_Selector, Connector_PinHeader_2.54mm:PinHeader_2x03_P2.54mm_Vertical, F.Cu at (63.2, 121.3)
- added J17: GND, Connector_PinHeader_2.54mm:PinHeader_1x01_P2.54mm_Vertical, F.Cu at (193.9, 116.5)
- added J18: GND, Connector_PinHeader_2.54mm:PinHeader_1x01_P2.54mm_Vertical, F.Cu at (162.0, 128.8)
- added J19: GND, Connector_PinHeader_2.54mm:PinHeader_1x01_P2.54mm_Vertical, F.Cu at (62.1, 30.1)
- added J2: PinHeader_Control, Connector_PinHeader_2.54mm:PinHeader_1x04_P2.54mm_Vertical, F.Cu at (109.3, 56.3)
- added J20: Conn_02x06_Odd_Even, Connector_PinHeader_2.54mm:PinHeader_2x06_P2.54mm_Vertical, F.Cu at (70.9, 111.2)
- added J22: Conn_02x04_Odd_Even, Connector_PinHeader_2.54mm:PinHeader_2x04_P2.54mm_Vertical, F.Cu at (87.1, 90.8)
- added J23: END_STOP_header, Connector_PinHeader_2.54mm:PinHeader_1x04_P2.54mm_Vertical, F.Cu at (108.5, 44.2)
- added J24: PinHeader_Control, Connector_PinHeader_2.54mm:PinHeader_1x04_P2.54mm_Vertical, F.Cu at (56.1, 144.5)
- added J25: Anemometer, TerminalBlock_Phoenix:TerminalBlock_Phoenix_MPT-0,5-4-2.54_1x04_P2.54mm_Horizontal, F.Cu at (49.1, 144.5)
- added J3: Motor, TerminalBlock_Phoenix:TerminalBlock_Phoenix_MKDS-3-2-5.08_1x02_P5.08mm_Horizontal, F.Cu at (192.0, 103.0)
- added J4: Stepper, TerminalBlock_Phoenix:TerminalBlock_Phoenix_MPT-0,5-4-2.54_1x04_P2.54mm_Horizontal, F.Cu at (49.0, 75.5)
- added J5: USR_BTN, TerminalBlock_Phoenix:TerminalBlock_Phoenix_MPT-0,5-2-2.54_1x02_P2.54mm_Horizontal, F.Cu at (99.0, 151.4)
- added J7: END_STOP_1_2, TerminalBlock_Phoenix:TerminalBlock_Phoenix_MPT-0,5-4-2.54_1x04_P2.54mm_Horizontal, F.Cu at (97.2, 31.2)
- added J8: USR_BTN, TerminalBlock_Phoenix:TerminalBlock_Phoenix_MPT-0,5-2-2.54_1x02_P2.54mm_Horizontal, F.Cu at (89.8, 151.4)
- added JP1: Jumper, Connector_PinHeader_2.54mm:PinHeader_1x02_P2.54mm_Vertical, F.Cu at (81.1, 35.7)
- added JP2: Jumper, Connector_PinHeader_2.54mm:PinHeader_1x02_P2.54mm_Vertical, F.Cu at (73.4, 49.6)
- added JP3: Jumper, Connector_PinHeader_2.54mm:PinHeader_1x02_P2.54mm_Vertical, F.Cu at (69.7, 52.1)
- added JP4: Jumper, Connector_PinHeader_2.54mm:PinHeader_1x02_P2.54mm_Vertical, F.Cu at (85.9, 61.1)
- added JP5: Jumper, Connector_PinHeader_2.54mm:PinHeader_1x02_P2.54mm_Vertical, F.Cu at (79.6, 61.8)
- added JP6: Jumper, Connector_PinHeader_2.54mm:PinHeader_1x02_P2.54mm_Vertical, F.Cu at (58.3, 62.2)
- added JP7: Jumper, Connector_PinHeader_2.54mm:PinHeader_1x02_P2.54mm_Vertical, F.Cu at (80.0, 69.9)
- added JP8: Jumper, Connector_PinHeader_2.54mm:PinHeader_1x02_P2.54mm_Vertical, F.Cu at (177.0, 132.0)
- added L1: L, Inductor_SMD:L_0603_1608Metric, B.Cu at (107.0, 109.8)
- added L2: L, Inductor_SMD:L_0603_1608Metric, B.Cu at (107.0, 106.8)
- added L3: L, Inductor_SMD:L_0603_1608Metric, B.Cu at (138.1, 104.3)
- added L4: L, Inductor_SMD:L_0603_1608Metric, B.Cu at (127.7, 104.2)
- added Q9: SI2302, Package_TO_SOT_SMD:SOT-23, B.Cu at (136.4, 133.8)
- added R1: 1k, Resistor_THT:R_Axial_DIN0207_L6.3mm_D2.5mm_P7.62mm_Horizontal, F.Cu at (152.5, 50.5)
- added R100: 1k, Resistor_SMD:R_0603_1608Metric, B.Cu at (134.2, 113.8)
- added R101: 1k, Resistor_SMD:R_0603_1608Metric, B.Cu at (137.6, 113.0)
- added R105: 10k, Resistor_THT:R_Axial_DIN0207_L6.3mm_D2.5mm_P7.62mm_Horizontal, F.Cu at (105.7, 69.6)
- added R12: 1K, Resistor_THT:R_Axial_DIN0207_L6.3mm_D2.5mm_P7.62mm_Horizontal, F.Cu at (134.0, 62.2)
- added R16: 100k, Resistor_THT:R_Axial_DIN0207_L6.3mm_D2.5mm_P7.62mm_Horizontal, F.Cu at (133.2, 74.0)
- added R2: 3.3K, Resistor_THT:R_Axial_DIN0207_L6.3mm_D2.5mm_P7.62mm_Horizontal, F.Cu at (171.6, 35.0)
- added R200: 470k, Resistor_THT:R_Axial_DIN0207_L6.3mm_D2.5mm_P7.62mm_Horizontal, F.Cu at (113.5, 96.0)
- added R201: 10k, Resistor_THT:R_Axial_DIN0207_L6.3mm_D2.5mm_P7.62mm_Horizontal, F.Cu at (157.2, 113.4)
- added R205: 10k, Resistor_THT:R_Axial_DIN0207_L6.3mm_D2.5mm_P7.62mm_Horizontal, F.Cu at (164.9, 108.4)
- added R21: 270, Resistor_THT:R_Axial_DIN0207_L6.3mm_D2.5mm_P7.62mm_Horizontal, F.Cu at (186.1, 85.7)
- added R27: 270, Resistor_THT:R_Axial_DIN0207_L6.3mm_D2.5mm_P7.62mm_Horizontal, F.Cu at (95.1, 66.2)
- added R28: 270, Resistor_THT:R_Axial_DIN0207_L6.3mm_D2.5mm_P7.62mm_Horizontal, F.Cu at (190.7, 131.8)
- added R29: 10k, Resistor_THT:R_Axial_DIN0207_L6.3mm_D2.5mm_P7.62mm_Horizontal, F.Cu at (80.7, 85.8)
- added R3: 3.3K, Resistor_THT:R_Axial_DIN0207_L6.3mm_D2.5mm_P7.62mm_Horizontal, F.Cu at (171.9, 42.7)
- added R30: 1k, Resistor_THT:R_Axial_DIN0207_L6.3mm_D2.5mm_P7.62mm_Horizontal, F.Cu at (76.4, 139.9)
- added R300: 10k, Resistor_THT:R_Axial_DIN0207_L6.3mm_D2.5mm_P7.62mm_Horizontal, F.Cu at (184.8, 40.2)
- added R301: 10k, Resistor_THT:R_Axial_DIN0207_L6.3mm_D2.5mm_P7.62mm_Horizontal, F.Cu at (188.4, 32.7)
- added R31: 1k, Resistor_THT:R_Axial_DIN0207_L6.3mm_D2.5mm_P7.62mm_Horizontal, F.Cu at (68.8, 136.8)
- added R32: 2.2k, Resistor_THT:R_Axial_DIN0207_L6.3mm_D2.5mm_P7.62mm_Horizontal, F.Cu at (89.3, 129.5)
- added R33: 1k, Resistor_SMD:R_0603_1608Metric, B.Cu at (131.5, 135.0)
- added R34: 10k, Resistor_SMD:R_0603_1608Metric, B.Cu at (135.4, 137.6)
- added R35: 0, Resistor_SMD:R_0603_1608Metric, B.Cu at (107.0, 118.7)
- added R36: 0, Resistor_SMD:R_0603_1608Metric, B.Cu at (107.0, 121.3)
- added R37: 0, Resistor_SMD:R_0603_1608Metric, B.Cu at (107.0, 123.1)
- added R38: 330, Resistor_SMD:R_0603_1608Metric, B.Cu at (144.1, 138.5)
- added R39: 0, Resistor_SMD:R_0603_1608Metric, B.Cu at (144.1, 135.0)
- added R4: 120, Resistor_THT:R_Axial_DIN0207_L6.3mm_D2.5mm_P7.62mm_Horizontal, F.Cu at (121.3, 47.9)
- added R40: 270, Resistor_THT:R_Axial_DIN0207_L6.3mm_D2.5mm_P7.62mm_Horizontal, F.Cu at (60.8, 50.6)
- added R41: 100, Resistor_THT:R_Axial_DIN0207_L6.3mm_D2.5mm_P7.62mm_Horizontal, F.Cu at (47.5, 61.7)
- added R42: 270, Resistor_THT:R_Axial_DIN0207_L6.3mm_D2.5mm_P7.62mm_Horizontal, F.Cu at (71.4, 57.5)
- added R43: 100, Resistor_THT:R_Axial_DIN0207_L6.3mm_D2.5mm_P7.62mm_Horizontal, F.Cu at (50.4, 70.0)
- added R48: 100, Resistor_THT:R_Axial_DIN0207_L6.3mm_D2.5mm_P7.62mm_Horizontal, F.Cu at (49.6, 50.1)
- added R5: 2.2K, Resistor_THT:R_Axial_DIN0207_L6.3mm_D2.5mm_P7.62mm_Horizontal, F.Cu at (139.6, 40.3)
- added R50: 10k, Resistor_THT:R_Axial_DIN0207_L6.3mm_D2.5mm_P7.62mm_Horizontal, F.Cu at (170.0, 124.4)
- added R51: 10k, Resistor_THT:R_Axial_DIN0207_L6.3mm_D2.5mm_P7.62mm_Horizontal, F.Cu at (181.4, 116.0)
- added R52: 10k, Resistor_THT:R_Axial_DIN0207_L6.3mm_D2.5mm_P7.62mm_Horizontal, F.Cu at (173.8, 127.6)
- added R6: 1K, Resistor_THT:R_Axial_DIN0207_L6.3mm_D2.5mm_P7.62mm_Horizontal, F.Cu at (133.9, 59.0)
- added R7: 1K, Resistor_THT:R_Axial_DIN0207_L6.3mm_D2.5mm_P7.62mm_Horizontal, F.Cu at (186.5, 60.0)
- added R8: 120, Resistor_THT:R_Axial_DIN0207_L6.3mm_D2.5mm_P7.62mm_Horizontal, F.Cu at (123.2, 66.2)
- added R9: 2.2K, Resistor_THT:R_Axial_DIN0207_L6.3mm_D2.5mm_P7.62mm_Horizontal, F.Cu at (126.3, 52.9)
- added RV2: R_Potentiometer, Potentiometer_THT:Potentiometer_Bourns_3266Y_Vertical, F.Cu at (186.2, 121.2)
- added SW1: SW_A, Button_Switch_THT:SW_PUSH_6mm_H8mm, F.Cu at (119.3, 69.1)
- added SW4: SW_B, Button_Switch_THT:SW_PUSH_6mm_H8mm, F.Cu at (102.6, 133.5)
- added SW5: SW_User, Button_Switch_THT:SW_PUSH_6mm_H8mm, F.Cu at (92.7, 133.4)
- added U1: PC817, Package_DIP:DIP-4_W7.62mm, F.Cu at (131.2, 44.5)
- added U11: L7805, Package_TO_SOT_THT:TO-220-3_Vertical, F.Cu at (78.4, 41.2)
- added U12: AMS1117-3.3, Package_TO_SOT_SMD:SOT-223-3_TabPin2, F.Cu at (85.9, 54.3)
- added U13: LM317_TO-220, Package_TO_SOT_THT:TO-220-3_Vertical, F.Cu at (55.7, 58.7)
- added U14: DS1307+, Package_DIP:DIP-8_W7.62mm, F.Cu at (92.0, 77.6)
- added U2: PC817, Package_DIP:DIP-4_W7.62mm, F.Cu at (116.1, 52.8)
- added U3: PC817, Package_DIP:DIP-4_W7.62mm, F.Cu at (186.4, 51.7)
- added U40: 74HC123, Package_DIP:DIP-16_W7.62mm_Socket, F.Cu at (150.4, 121.0)
- added U41: LM358, Package_DIP:DIP-8_W7.62mm_Socket, F.Cu at (177.8, 121.1)
- added U6: NRF24L01_Breakout, RF_Module:nRF24L01_Breakout, F.Cu at (58.5, 111.3)
- added U8: NEO-M8M, RF_GPS:ublox_NEO, B.Cu at (134.1, 122.7)
- added U9: ATmega328P-P, Package_DIP:DIP-28_W7.62mm_Socket, F.Cu at (84.2, 123.8)
- added Y2: 16MHz, Crystal:Crystal_AT310_D3.0mm_L10.0mm_Horizontal, F.Cu at (88.7, 78.2)
- C4: value 100n -> 100nF; footprint Capacitor_THT:C_Radial_D4.0mm_H5.0mm_P1.50mm -> Capacitor_THT:C_Radial_D5.0mm_H11.0mm_P2.00mm
- C5: value 22pF -> 100nF; footprint Capacitor_THT:C_Disc_D4.7mm_W2.5mm_P5.00mm -> Capacitor_SMD:C_0603_1608Metric
- C8: value 20F -> 100nF; footprint Capacitor_THT:C_Radial_D10.0mm_H20.0mm_P5.00mm -> Capacitor_THT:C_Radial_D5.0mm_H11.0mm_P2.00mm
- J10: value 132134 -> PinHeader_Control; footprint Connector_Coaxial:SMA_Molex_73251-1153_EdgeMount_Horizontal -> Connector_PinHeader_2.54mm:PinHeader_1x04_P2.54mm_Vertical
- J11: value SPI_Programming -> Conn_02x05_Odd_Even
- J6: value GND -> Wind; footprint Connector_PinHeader_2.54mm:PinHeader_1x01_P2.54mm_Vertical -> TerminalBlock_Phoenix:TerminalBlock_Phoenix_MPT-0,5-2-2.54_1x02_P2.54mm_Horizontal
- J9: value Haeder_LED -> Analog_Position; footprint Connector_PinHeader_2.54mm:PinHeader_2x01_P2.54mm_Vertical -> TerminalBlock_Phoenix:TerminalBlock_Phoenix_MPT-0,5-3-2.54_1x03_P2.54mm_Horizontal
- R11, R14, R15: value 470 -> 120
- R20: value 470 -> 270
- R25: value 2.7k -> 1k
- RV1: value V_Selector -> R_Potentiometer; footprint Potentiometer_THT:Potentiometer_Bourns_3386C_Horizontal -> Potentiometer_THT:Potentiometer_Alps_RK163_Single_Horizontal
- SW2: value SW_A -> SW_B
- U7: value GK9501 -> AS193-73; footprint RF_GPS:ublox_NEO -> Package_TO_SOT_SMD:SOT-23-6; moved to B.Cu
- moved C8 143.8 mm to (84.4, 41.3), turned to 90 degrees
- moved J10 135.1 mm to (55.8, 75.5), turned to 0 degrees
- moved J9 121.8 mm to (198.0, 39.0), turned to 90 degrees
- moved C5 117.9 mm to (167.1, 112.6), turned to 90 degrees
- moved J6 116.3 mm to (184.0, 150.7)
- moved U7 64.8 mm to (128.1, 137.1)
- moved C6 59.4 mm to (100.4, 109.7), turned to 90 degrees
- moved C4 55.2 mm to (166.2, 121.0), turned to 180 degrees
- moved RV1 49.8 mm to (153.9, 154.6)
- moved J11 46.0 mm to (73.4, 101.0), turned to 180 degrees
- moved Y1 42.9 mm to (95.7, 99.7), turned to -90 degrees
- moved R22 40.2 mm to (198.9, 108.8), turned to -90 degrees
- moved D8 38.8 mm to (195.0, 108.7), turned to 180 degrees
- moved R23 27.1 mm to (198.4, 91.9), turned to 90 degrees
- moved D9 24.5 mm to (194.8, 92.1), turned to 180 degrees
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Connections:
- C4 pad 1: /+VCC_Wind -> +5V
- C5 pad 1: GND -> Net-(U41B-+)
- C5 pad 2: /Crystal/XTAl_1 -> GND
- C6 pad 2: /Crystal/XTAl_2 -> /Crystal/XTAl_1
- D10 pad 1: /IN_A -> /Motors/IN_A
- D10 pad 2: Net-(D10-A) -> /MCU/PD5-D5~
- D11 pad 1: /IN_B -> /Motors/IN_B
- D11 pad 2: Net-(D11-A) -> /MCU/PD4-D4
- D13 pad 1: /ENABLE -> /Motors/ENABLE
- D13 pad 2: Net-(D13-A) -> /MCU/PD3-D3-(INT1)~
- D6 pad 2: /IN_B -> /Motors/IN_B
- J10 pad 1: Net-(J10-In) -> /MCU/PB0-D8
- J10 pad 2: GND -> /MCU/PB1-D9~
- J11 pad 1: /MOSI -> Net-(J11-Pin_1)
- J11 pad 10: GND -> /MCU/PB1-D9~
- J11 pad 2: +5V -> /MCU/CLK
- J11 pad 3: +5V -> Net-(J11-Pin_3)
- J11 pad 4: GND -> /MCU/MISO
- J11 pad 5: /RST -> Net-(J11-Pin_5)
- J11 pad 6: GND -> /MCU/MOSI
- J11 pad 7: /SCK -> Net-(J11-Pin_7)
- J11 pad 8: GND -> /MCU/PB2-D10~
- J11 pad 9: /MISO -> Net-(J11-Pin_9)
- J6 pad 1: GND -> Net-(J13-Pin_1)
- J9 pad 1: +5V -> GND
- Q6 pad 2: /IN_A -> /Motors/IN_A
- Q7 pad 2: /IN_B -> /Motors/IN_B
- R11 pad 2: /IN_B -> /Motors/IN_B
- R14 pad 1: /IN_B -> /Motors/IN_B
- R15 pad 2: /IN_A -> /Motors/IN_A
- R18 pad 1: /IN_A -> /Motors/IN_A
- R19 pad 1: /IN_B -> /Motors/IN_B
- RV1 pad 1: /+VCC_Wind -> GND
- RV1 pad 2: Net-(U2A--) -> /MCU/PC1-A1
- RV1 pad 3: GND -> +5V
- SW2 pad 1: /IN_A -> /Motors/IN_B
- SW3 pad 1: /ENABLE -> Net-(J23-Pin_1)
- U7 pad 1: unconnected-(U7-NC-Pad1) -> Net-(U7-RF1)
- U7 pad 2: unconnected-(U7-NC-Pad2) -> GND_GNSS
- U7 pad 3: /GNSS/PPS -> Net-(U7-RF2)
- U7 pad 4: unconnected-(U7-EXTINT3-Pad4) -> /GNSS/~{INTERNAL_ANTENNA}
- U7 pad 5: (no net) -> Net-(U7-RFC)
- U7 pad 6: unconnected-(U7-EXTINT0-Pad6) -> Net-(Q9-D)
Routing:
- net /IN_A: track 163.5 -> 0.00 mm
- net +5V: track 47.6 -> 202.8 mm, vias 0 -> 1
- net /IN_B: track 138.2 -> 0.00 mm
- net /+VCC_Wind: track 112.2 -> 0.00 mm, vias 1 -> 0
- net /Motors/IN_A: track 1.51 -> 113.4 mm
- net Net-(J23-Pin_1): track 0.00 -> 82.0 mm, vias 0 -> 2
- net +VCap: track 0.00 -> 77.1 mm, vias 0 -> 3
- net /V_{A_{2}}: track 0.00 -> 64.4 mm, vias 0 -> 2
- net /Motors/IN_B: track 18.6 -> 77.8 mm
- net /Anemometer/SDA: track 0.00 -> 55.7 mm, vias 0 -> 2
- net /Anemometer/SCL: track 0.00 -> 54.2 mm, vias 0 -> 2
- net Net-(D4-K): track 79.7 -> 133.3 mm
- net Net-(D10-A): track 47.1 -> 0.00 mm
- net /MCU/MOSI: track 0.00 -> 45.0 mm, vias 0 -> 3
- net /MCU/MISO: track 0.00 -> 44.8 mm, vias 0 -> 1
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- added copper zone on B.Cu, net GND_GNSS
- added copper zone on F.Cu, net GND_GNSS
Other:
- board size 167.4 x 98.3 mm -> 173.6 x 133.6 mm
- board text added: "+3.3V_ON"
- board text added: "+5V_EN"
- board text added: "+5V_ICC"
- board text added: "+5V_ON"
- board text added: "16MHz"
- board text added: "ANALOG_POS"
- board text added: "AVR_ISP"
- board text added: "END_1"
- board text added: "END_2"
- board text added: "LED_EN"
- board text added: "LED_ON"
- board text added: "Motor"
- board text added: "RESET"
- board text added: "Tracker solaire - CREPP V1.0"
- board text added: "USER"
- board text added: "VCAP_ON"
- board text removed: "CFT - V1"
- board text removed: "Tracker solaire - CREPP Carte de contrôle moteur V1.0"
