File: Hardware/Tracker.kicad_sch (KiCad schematic)
At the start: 27 parts, among them J1 Battery, J11 SPI_Programming, J4 RX, J5 TX, J6 GND, J7 GND, J8 GND, J9 Haeder_LED, U1 L7805, U2 ATmega328P-P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

Commit message: update of directory
Connections:
- net Motors/EN_MOTOR: now reaches U2.23 (PC0)
- net Motors/IN2_MOTOR: now reaches U2.24 (PC1)
- net Motors/IN1_MOTOR: now reaches U2.25 (PC2)
- net WIND/Wind_interrupt: now reaches U2.5 (PD3)
- net WIND/OUT renamed WIND/RAW_DATA
Other:
- sheet Motors ports: added EN_MOTOR, IN1_MOTOR, IN2_MOTOR; removed none
- sheet WIND ports: added RAW_DATA, Wind_interrupt; removed OUT
- note added: "Prise en compte 24V"
Changed lines of the file:
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@@
+    (stroke (width 0) (type default))
+  )
+  (wire (pts (xy 142.24 90.17) (xy 168.91 90.17))
     (stroke (width 0) (type default))
   )
@@
     (stroke (width 0) (type default))
   )
+  (wire (pts (xy 142.24 113.03) (xy 161.29 113.03))
+    (stroke (width 0) (type default))
+  )
   (wire (pts (xy 129.54 53.34) (xy 128.27 53.34))
     (stroke (width 0) (type default))
@@
     (stroke (width 0) (type default))
   )
+  (wire (pts (xy 142.24 85.09) (xy 168.91 85.09))
+    (stroke (width 0) (type default))
+  )
   (wire (pts (xy 237.49 96.52) (xy 238.76 96.52))
     (stroke (width 0) (type default))
@@
     (stroke (width 0) (type default))
   )
+  (wire (pts (xy 142.24 87.63) (xy 168.91 87.63))
+    (stroke (width 0) (type default))
+  )
   (wire (pts (xy 147.32 40.64) (xy 147.32 43.18))
     (stroke (width 0) (type default))
@@
     (stroke (width 0) (type default))
   )
-  (wire (pts (xy 142.24 110.49) (xy 162.56 110.49))
+  (wire (pts (xy 142.24 110.49) (xy 161.29 110.49))
     (stroke (width 0) (type default))
   )
@@
   (wire (pts (xy 34.29 29.21) (xy 34.29 43.18))
     (stroke (width 0) (type default))
+  )
+  (text "Prise en compte 24V\n" (at 133.35 20.32 0)
+    (effects (font (size 1.27 1.27)) (justify left bottom))
   )
   (text "Pin 3 is routed to +5V but pin must be cutted" (at 224.79 101.6 0)
@@
     )
   )
-  (sheet (at 162.56 107.95) (size 12.7 5.08)
+  (sheet (at 161.29 107.95) (size 16.51 7.62) (fields_autoplaced)
     (stroke (width 0.1524) (type solid))
     (fill (color 0 0 0 0.0000))
-    (property "Sheetname" "WIND" (at 176.53 111.76 0)
+    (property "Sheetname" "WIND" (at 161.29 107.2384 0)
       (effects (font (size 1.27 1.27)) (justify left bottom))
     )
-    (property "Sheetfile" "WIND.kicad_sch" (at 162.56 116.1546 0)
+    (property "Sheetfile" "WIND.kicad_sch" (at 161.29 116.1546 0)
       (effects (font (size 1.27 1.27)) (justify left top) hide)
     )
-    (pin "OUT" output (at 162.56 110.49 180)
+    (pin "Wind_interrupt" output (at 161.29 113.03 180)
+      (effects (font (size 1.27 1.27)) (justify left))
+    )
+    (pin "RAW_DATA" output (at 161.29 110.49 180)
       (effects (font (size 1.27 1.27)) (justify left))
     )
@@
     )
   )
-  (sheet (at 22.86 106.68) (size 25.4 26.67) (fields_autoplaced)
+  (sheet (at 168.91 83.82) (size 36.83 16.51) (fields_autoplaced)
     (stroke (width 0.1524) (type solid))
     (fill (color 0 0 0 0.0000))
-    (property "Sheetname" "Motors" (at 22.86 105.9684 0)
+    (property "Sheetname" "Motors" (at 168.91 83.1084 0)
       (effects (font (size 1.27 1.27)) (justify left bottom))
     )
-    (property "Sheetfile" "Motors.kicad_sch" (at 22.86 133.9346 0)
+    (property "Sheetfile" "Motors.kicad_sch" (at 168.91 100.9146 0)
       (effects (font (size 1.27 1.27)) (justify left top) hide)
     )
-    (instances
+    (pin "IN1_MOTOR" input (at 168.91 90.17 180)
+      (effects (font (size 1.27 1.27)) (justify left))
+    )
+    (pin "EN_MOTOR" input (at 168.91 85.09 180)
+      (effects (font (size 1.27 1.27)) (justify left))
+    )
+    (pin "IN2_MOTOR" input (at 168.91 87.63 180)
+      (effects (font (size 1.27 1.27)) (justify left))
+    )
+    (instances
