File: Hardware/Modules/WIND.kicad_sch (KiCad schematic)
At the start: 14 parts, among them J9 Wind, U3 LM358, U4 74HC123

Commit message: Update of PCB
Parts:
- added D18: LED, LED_THT:LED_D3.0mm, symbol Device:LED
- added J13: RAW_data_Wind, Connector_PinHeader_2.54mm:PinHeader_1x01_P2.54mm_Vertical, symbol Connector:Conn_01x01_Pin
- added JP8: Jumper, Connector_PinHeader_2.54mm:PinHeader_1x02_P2.54mm_Vertical, symbol Jumper:Jumper_2_Bridged
- added R28: 270, Resistor_THT:R_Axial_DIN0207_L6.3mm_D2.5mm_P7.62mm_Horizontal, symbol Device:R
- added unit 2 of U40
- added unit 2 of U41
- C2: renamed from C3; footprint Capacitor_THT:C_Rect_L7.0mm_W2.0mm_P5.00mm -> Capacitor_THT:C_Radial_D5.0mm_H11.0mm_P2.00mm
- C3: renamed from C4; footprint Capacitor_THT:C_Rect_L7.0mm_W2.0mm_P5.00mm -> Capacitor_SMD:C_0603_1608Metric
- C4: renamed from C5; footprint Capacitor_THT:C_Rect_L7.0mm_W2.0mm_P5.00mm -> Capacitor_THT:C_Radial_D5.0mm_H11.0mm_P2.00mm
- C5: renamed from C6; footprint Capacitor_THT:C_Rect_L7.0mm_W2.0mm_P5.00mm -> Capacitor_SMD:C_0603_1608Metric
- J6: renamed from J9; footprint TerminalBlock_Phoenix:TerminalBlock_Phoenix_MKDS-1,5-2-5.08_1x02_P5.08mm_Horizontal -> TerminalBlock_Phoenix:TerminalBlock_Phoenix_MPT-0,5-2-2.54_1x02_P2.54mm_Horizontal
- renumbered R3 to R200, R5 to R201, R4 to R205, R6 to R50, R7 to R51, R8 to R52, RV1 to RV2, U4 to U40, U3 to U41
Connections:
- net GND: now also R28.2
- net Wind_interrupt: now also JP8.1 (A)
- net at C5.1, R201.2: now also U41.5 (+); no longer R50.1
- net RAW_DATA: no longer names the net of J6.1 (Pin_1), R200.2, U40.2 (B)
- net RAW_DATA: now also J13.1 (Pin_1)
- new net: D18.1 (K), R28.1
- new net: D18.2 (A), JP8.2 (B)
- new net: R50.1, U41.6 (-), U41.7
- no-connect marks 2 -> 9
Other:
- title: (none) -> Wind handler
- moved on the sheet: R50, R51, R52, RV2, U41A
