File: Hardware/V1_THT/Tracker.kicad_sch (KiCad schematic)
At the start: 7 parts

Commit message: update of directory
Other:
- sheet Motors: file ../../../Electronique/Kicad/Motor_Control/Motor_Control.kicad_sch -> Modules/Motor_Control.kicad_sch
Changed lines of the file:
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@@
 			)
 		)
-		(property "Sheetfile" "../../../Electronique/Kicad/Motor_Control/Motor_Control.kicad_sch"
+		(property "Sheetfile" "Modules/Motor_Control.kicad_sch"
 			(at 176.53 133.9346 0)
 			(effects
