File: Hardware/V1_THT/Tracker.kicad_pcb (KiCad board)
At the start: 2 copper layers, 164.3 x 134.9 mm, 181 parts, among them J1 +24V, J10 PinHeader_Control, J100 132134, J11 Conn_02x05_Odd_Even, J12 Conn_02x06_Odd_Even, J13 RAW_data_Wind, J14 OLED_SOCKET, J15 SPI_Programming, J16 I2C_Selector, J17 GND, J18 GND, J19 GND, J2 PinHeader_Control, J20 Conn_02x06_Odd_Even, J22 Conn_02x04_Odd_Even, J23 END_STOP_header, J24 PinHeader_Control, J25 Anemometer, J3 Motor, J4 Stepper, J5 USR_BTN, J6 Wind, J7 END_STOP_1_2, J8 USR_BTN, J9 Analog_Position, Q1 IRF4905, Q2 IRF4905, Q3 IRF4905, Q4 IRF520, Q5 IRF520, Q6 2N7000, Q7 2N7000, Q9 SI2302, SW1 SW_A, SW2 SW_B, SW3 SW_E, SW4 SW_B, SW5 SW_User, U1 PC817, U11 L7805, U12 AMS1117-3.3, U13 LM317_TO-220, U14 DS1307+, U2 PC817, U3 PC817, U4 PC817, U40 74HC123, U41 LM358, U5 PC817, U6 NRF24L01_Breakout, U7 AS193-73, U8 NEO-M8M, U9 ATmega328P-P, Y1 16MHz, Y2 16MHz

Commit message: Update of PCB
Parts:
- moved H3 215.1 mm to (-14.7, 74.8), turned to -90 degrees
Changed lines of the file:
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@@
 	(footprint "MountingHole:MountingHole_3mm"
 		(layer "F.Cu")
-		(at 196.19 32.13)
+		(at -14.65 74.77 -90)
 		(descr "Mounting Hole 3mm, no annular")
 		(tags "mounting hole 3mm no annular")
 		(property "Reference" "H3"
-			(at 1.36 5 0)
+			(at 1.36 5 90)
 			(layer "F.SilkS")
 			(hide yes)
@@
 		)
 		(property "Value" "MountingHole"
-			(at 0 4 0)
+			(at 0 4 90)
 			(layer "F.Fab")
 			(effects
@@
 		)
 		(property "Footprint" "MountingHole:MountingHole_3mm"
-			(at 0 0 0)
+			(at 0 0 -90)
 			(unlocked yes)
 			(layer "F.Fab")
@@
 		)
 		(property "Datasheet" ""
-			(at 0 0 0)
+			(at 0 0 -90)
 			(unlocked yes)
 			(layer "F.Fab")
@@
 		)
 		(property "Description" ""
-			(at 0 0 0)
+			(at 0 0 -90)
 			(unlocked yes)
 			(layer "F.Fab")
@@
 		)
 		(fp_text user "${REFERENCE}"
-			(at 0 0 0)
+			(at 0 0 90)
 			(layer "F.Fab")
 			(effects
@@
 		)
 		(pad "" np_thru_hole circle
-			(at 0 0)
+			(at 0 0 270)
 			(size 3 3)
 			(drill 3)
 			(layers "*.Cu" "*.Mask")
 		)
+		(model "/home/nico/Documents/Electronique/Kicad/Libraries_3D_Footprints/Steppers/TB6600/TB6600.STEP"
+			(offset
+				(xyz 0 0 20)
+			)
+			(scale
+				(xyz 1 1 1)
+			)
+			(rotate
+				(xyz 90 0 0)
+			)
+		)
 	)
