File: Hardware/V2_CMS/Tracker.kicad_pcb (KiCad board)
At the start: 2 copper layers, 172 parts, among them J1 Wind, J10 SPI_Programming, J11 USR_BTN, J12 GND, J13 GND, J14 GND, J15 PinHeader_Control, J16 Stepper, J17 PinHeader_Control, J18 Anemometer, J19 USR_BTN, J2 RAW_data_Wind, J3 132134, J4 PinHeader_Control, J5 Control, J6 +24V, J7 Motor, J8 I2C_Selector, J9 OLED_SOCKET, Q1 SI2302, Q2 IRF4905, Q3 2N7000, Q4 IRF4905, Q5 IRF520, Q6 IRF4905, Q7 IRF520, Q8 2N7000, SW1 SW_E, SW2 SW_B, SW3 SW_A, SW4 SW_B, SW5 SW_User, U1 LM358, U10 L7805, U11 AMS1117-3.3, U12 LM317_TO-220, U13 DS1307+, U14 NRF24L01_Breakout, U15 ATmega328P-A, U2 74HC123, U3 NEO-M8M, U4 AS193-73, U5 PC817, U6 PC817, U7 PC817, U8 PC817, U9 PC817, Y1 16MHz, Y2 32kHz

Commit message: update of directory
Parts:
- removed C8: 100nF, Capacitor_SMD:C_0603_1608Metric
- removed F1: Fuse, Fuse:Fuseholder_Cylinder-5x20mm_Schurter_0031_8201_Horizontal_Open
- removed H5, H6, H7, H8: MountingHole, MountingHole:MountingHole_3mm
- removed J13, J14: GND, Connector_PinHeader_2.54mm:PinHeader_1x01_P2.54mm_Vertical
- removed J15, J17: PinHeader_Control, Connector_PinHeader_2.54mm:PinHeader_1x04_P2.54mm_Vertical
- removed JP1, JP3, JP4, JP5, JP6, JP7: Jumper, Connector_PinHeader_2.54mm:PinHeader_1x02_P2.54mm_Vertical
- added C23: 100nF, Capacitor_SMD:C_0603_1608Metric, F.Cu at (195.7, 124.9)
- added C24: 100nF, Capacitor_SMD:C_0603_1608Metric, F.Cu at (195.8, 121.1)
- added C25: 330pF, Capacitor_SMD:C_0603_1608Metric, B.Cu at (115.5, 153.8)
- added C26: 330pF, Capacitor_SMD:C_0603_1608Metric, B.Cu at (117.9, 156.1)
- added C27: 100nF, Capacitor_SMD:C_0603_1608Metric, B.Cu at (114.9, 89.7)
- added C28: 4.7u, Capacitor_SMD:C_0603_1608Metric, F.Cu at (112.9, 72.8)
- added C29: 100nF, Capacitor_SMD:C_0603_1608Metric, F.Cu at (144.6, 115.0)
- added C30: 100nF, Capacitor_SMD:C_0603_1608Metric, B.Cu at (148.4, 66.2)
- added C31: XX, Capacitor_SMD:C_0603_1608Metric, F.Cu at (118.9, 72.1)
- added C32: XX, Capacitor_SMD:C_0603_1608Metric, F.Cu at (118.9, 74.6)
- added C33: 220uF, Capacitor_SMD:CP_Elec_6.3x7.7, B.Cu at (166.4, 92.6)
- added C34: 120pF, Capacitor_SMD:C_0603_1608Metric, B.Cu at (116.9, 145.9)
- added C35: 1nF, Capacitor_SMD:C_0603_1608Metric, B.Cu at (105.0, 131.9)
- added C36: 100nF, Capacitor_SMD:C_0603_1608Metric, B.Cu at (105.0, 134.8)
- added C37: 100nF, Capacitor_SMD:C_0603_1608Metric, B.Cu at (184.7, 82.0)
- added C38: 100nF, Capacitor_SMD:C_0603_1608Metric, F.Cu at (206.6, 114.2)
- added C39: 100nF, Capacitor_SMD:C_0603_1608Metric, F.Cu at (186.2, 107.9)
- added D21: LED, LED_SMD:LED_0603_1608Metric, F.Cu at (157.4, 140.4)
- added D22: 1N4148, Diode_SMD:D_SOD-323, B.Cu at (123.3, 66.6)
- added D23: SS34, Diode_SMD:D_SMA, B.Cu at (176.6, 92.5)
- added D24: GNSS_USB, LED_SMD:LED_0603_1608Metric, F.Cu at (115.5, 122.7)
- added D25: LED_USB, LED_SMD:LED_0603_1608Metric, F.Cu at (199.6, 121.3)
- added D26: TX_LED, LED_SMD:LED_0603_1608Metric, F.Cu at (191.2, 124.0)
- added D27: RX_LED, LED_SMD:LED_0603_1608Metric, F.Cu at (192.9, 124.0)
- added D28: LED_EXT_ANTENNA, LED_SMD:LED_0603_1608Metric, F.Cu at (115.5, 124.6)
- added D29: ZENER_5.6V, Diode_SMD:D_MiniMELF, B.Cu at (165.4, 87.3)
- added D30: 1N4148, Diode_SMD:D_SOD-323, B.Cu at (190.6, 65.5)
- added D31: ZENER_3.6V, Diode_SMD:D_MiniMELF, B.Cu at (134.9, 114.6)
- added D32: 1N4148, Diode_SMD:D_SOD-323, B.Cu at (195.3, 78.2)
- added D33: LED, LED_SMD:LED_0603_1608Metric, F.Cu at (188.5, 90.4)
- added D34: GNSS_BATT, LED_SMD:LED_0603_1608Metric, F.Cu at (115.6, 116.8)
- added D35: 1N4148, Diode_SMD:D_SOD-323, B.Cu at (126.5, 82.0)
- added D36: 1N4148, Diode_SMD:D_SOD-323, B.Cu at (129.6, 128.5)
- added G***: LOGO, LOGO, F.Cu at (195.1, 154.6)
- added HS5: Heatsink, HeatSink:HeastSink_MOSFET_15mm_10mm_20mm, F.Cu at (198.5, 51.7)
- added IC1: L6208, Package_SO:ST_PowerSSO-36_SlugDown_ThermalVias, F.Cu at (122.5, 49.4)
- added J20: 132415, Connector_Coaxial:SMA_Molex_73251-1153_EdgeMount_Horizontal, F.Cu at (100.4, 90.2)
- added J21: USR_BTN_1, TerminalBlock_Phoenix:TerminalBlock_Phoenix_MPT-0,5-2-2.54_1x02_P2.54mm_Horizontal, F.Cu at (139.4, 154.7)
- added J22: Stepper_Pos, TerminalBlock_Phoenix:TerminalBlock_Phoenix_MPT-0,5-2-2.54_1x02_P2.54mm_Horizontal, F.Cu at (138.1, 54.6)
- added J23: END_STOP_1, TerminalBlock_Phoenix:TerminalBlock_Phoenix_MPT-0,5-2-2.54_1x02_P2.54mm_Horizontal, F.Cu at (187.7, 25.3)
- added J25: END_STOP_1, TerminalBlock_Phoenix:TerminalBlock_Phoenix_MPT-0,5-2-2.54_1x02_P2.54mm_Horizontal, F.Cu at (178.5, 25.3)
- added J26: +24V, Connector_Phoenix_MSTB:PhoenixContact_MSTBA_2,5_2-G-5,08_1x02_P5.08mm_Horizontal, F.Cu at (108.2, 29.1)
- added J27: EN_LED, TerminalBlock_Phoenix:TerminalBlock_Phoenix_MPT-0,5-2-2.54_1x02_P2.54mm_Horizontal, F.Cu at (194.7, 25.2)
- added J28: SW_EN, TerminalBlock_Phoenix:TerminalBlock_Phoenix_MPT-0,5-2-2.54_1x02_P2.54mm_Horizontal, F.Cu at (206.5, 41.4)
- added J29: EXT_SW_A, TerminalBlock_Phoenix:TerminalBlock_Phoenix_MPT-0,5-2-2.54_1x02_P2.54mm_Horizontal, F.Cu at (206.5, 34.3)
- added J30: EXT_SW_B, TerminalBlock_Phoenix:TerminalBlock_Phoenix_MPT-0,5-2-2.54_1x02_P2.54mm_Horizontal, F.Cu at (206.2, 27.2)
- added J31: Motor_Control_Pull_Up, TerminalBlock_Phoenix:TerminalBlock_Phoenix_MPT-0,5-3-2.54_1x03_P2.54mm_Horizontal, F.Cu at (101.4, 75.1)
- added J32: Motor_Control, TerminalBlock_Phoenix:TerminalBlock_Phoenix_MPT-0,5-3-2.54_1x03_P2.54mm_Horizontal, F.Cu at (101.7, 65.8)
- added J33: Fuse, Connector_Phoenix_MSTB:PhoenixContact_MSTBA_2,5_2-G-5,08_1x02_P5.08mm_Horizontal, F.Cu at (145.8, 31.2)
- added J35: LDR, TerminalBlock_Phoenix:TerminalBlock_Phoenix_MPT-0,5-2-2.54_1x02_P2.54mm_Horizontal, F.Cu at (204.7, 71.6)
- added J36: SWITCH_POWER, TerminalBlock_Phoenix:TerminalBlock_Phoenix_MPT-0,5-2-2.54_1x02_P2.54mm_Horizontal, F.Cu at (204.7, 78.2)
- added J37: Micro_SD_Card, Connector_Card:microSD_HC_Hirose_DM3D-SF, F.Cu at (203.6, 105.6)
- added JP10: Jumper_2_Open, Connector_PinHeader_1.27mm:PinHeader_1x02_P1.27mm_Vertical, F.Cu at (150.6, 109.3)
- added JP11: Jumper_2_Open, Connector_PinHeader_1.27mm:PinHeader_1x02_P1.27mm_Vertical, F.Cu at (149.3, 109.3)
- added JP12: Jumper_2_Open, Connector_PinHeader_1.27mm:PinHeader_1x02_P1.27mm_Vertical, F.Cu at (148.0, 109.3)
- added JP13: Jumper_2_Open, Connector_PinHeader_1.27mm:PinHeader_1x02_P1.27mm_Vertical, F.Cu at (144.9, 112.6)
- added JP14: Jumper_2_Open, Connector_PinHeader_1.27mm:PinHeader_1x02_P1.27mm_Vertical, F.Cu at (144.8, 118.6)
- added JP15: Jumper_2_Open, Connector_PinHeader_1.27mm:PinHeader_1x02_P1.27mm_Vertical, F.Cu at (144.7, 120.1)
- added JP16: Jumper_2_Open, Connector_PinHeader_1.27mm:PinHeader_1x02_P1.27mm_Vertical, F.Cu at (148.0, 124.5)
- added JP17: Jumper_2_Open, Connector_PinHeader_1.27mm:PinHeader_1x02_P1.27mm_Vertical, F.Cu at (149.3, 124.5)
- added JP18: Jumper_2_Open, Connector_PinHeader_1.27mm:PinHeader_1x02_P1.27mm_Vertical, F.Cu at (150.6, 124.5)
- added JP19: Jumper_2_Open, Connector_PinHeader_1.27mm:PinHeader_1x02_P1.27mm_Vertical, F.Cu at (151.8, 124.5)
- added JP20: Jumper_2_Open, Connector_PinHeader_1.27mm:PinHeader_1x02_P1.27mm_Vertical, F.Cu at (153.1, 124.5)
- added JP21: Jumper_2_Open, Connector_PinHeader_1.27mm:PinHeader_1x02_P1.27mm_Vertical, F.Cu at (154.4, 124.5)
- added JP22: Jumper_2_Open, Connector_PinHeader_1.27mm:PinHeader_1x02_P1.27mm_Vertical, F.Cu at (155.7, 124.5)
- added JP23: Jumper_2_Open, Connector_PinHeader_1.27mm:PinHeader_1x02_P1.27mm_Vertical, F.Cu at (156.9, 124.5)
- added JP24: Jumper_2_Open, Connector_PinHeader_1.27mm:PinHeader_1x02_P1.27mm_Vertical, F.Cu at (161.7, 109.3)
- added JP25: Jumper_2_Open, Connector_PinHeader_1.27mm:PinHeader_1x02_P1.27mm_Vertical, F.Cu at (160.4, 109.3)
- added JP26: Jumper_2_Open, Connector_PinHeader_1.27mm:PinHeader_1x02_P1.27mm_Vertical, F.Cu at (154.4, 109.3)
- added JP27: Jumper_2_Open, Connector_PinHeader_1.27mm:PinHeader_1x02_P1.27mm_Vertical, F.Cu at (155.5, 109.3)
- added JP28: Jumper_2_Open, Connector_PinHeader_1.27mm:PinHeader_1x02_P1.27mm_Vertical, F.Cu at (156.9, 109.3)
- added JP29: Jumper, Connector_PinHeader_2.54mm:PinHeader_1x02_P2.54mm_Vertical, F.Cu at (184.9, 31.5)
- added JP9: Jumper_2_Open, Connector_PinHeader_1.27mm:PinHeader_1x02_P1.27mm_Vertical, F.Cu at (151.8, 109.3)
- added L10: MPZ1608, Inductor_SMD:L_0603_1608Metric, B.Cu at (113.8, 84.0)
- added L11: MPZ1608, Inductor_SMD:L_0603_1608Metric, B.Cu at (187.1, 84.1)
- added L12: MPZ1608, Inductor_SMD:L_0603_1608Metric, F.Cu at (-24.6, 22.9)
- added L13: MPZ1608, Inductor_SMD:L_0603_1608Metric, B.Cu at (170.6, 88.2)
- added L14: MPZ1608, Inductor_SMD:L_0603_1608Metric, B.Cu at (131.3, 111.8)
- added L5: 33nH, Inductor_SMD:L_Wuerth_HCI-5040, B.Cu at (175.3, 87.0)
- added L6: 56nH, Inductor_SMD:L_0603_1608Metric, B.Cu at (115.5, 151.3)
- added L7: MPZ1608, Inductor_SMD:L_0603_1608Metric, B.Cu at (170.4, 85.1)
- added L8: MPZ1608, Inductor_SMD:L_0603_1608Metric, B.Cu at (181.8, 95.1)
- added L9: 39nH, Inductor_SMD:L_0603_1608Metric, B.Cu at (114.2, 146.7)
- added Q10: CJ3401, Package_TO_SOT_SMD:SOT-23, B.Cu at (126.1, 117.5)
- added Q11: 2N7002, Package_TO_SOT_SMD:SOT-23, B.Cu at (132.5, 143.1)
- added Q9: 2N7002, Package_TO_SOT_SMD:SOT-23, B.Cu at (190.8, 61.3)
- added R100: 10k, Resistor_SMD:R_0603_1608Metric, B.Cu at (144.0, 77.7)
- added R101: 10k, Resistor_SMD:R_0603_1608Metric, B.Cu at (151.2, 108.3)
- added R102: 0, Resistor_SMD:R_0603_1608Metric, F.Cu at (136.2, 84.0)
- added R103: 0, Resistor_SMD:R_0603_1608Metric, F.Cu at (132.2, 84.1)
- added R104: 0, Resistor_SMD:R_0603_1608Metric, F.Cu at (109.5, 84.0)
- added R105: 0, Resistor_SMD:R_0603_1608Metric, F.Cu at (124.9, 102.5)
- added R106: 0, Resistor_SMD:R_0603_1608Metric, F.Cu at (122.2, 124.6)
- added R107: 0, Resistor_SMD:R_0603_1608Metric, F.Cu at (136.1, 143.0)
- added R54: 270, Resistor_SMD:R_0603_1608Metric, F.Cu at (191.2, 120.7)
- added R55: 270, Resistor_SMD:R_0603_1608Metric, F.Cu at (192.9, 120.7)
- added R56: 100k, Resistor_SMD:R_0603_1608Metric, B.Cu at (109.4, 151.3)
- added R57: 10k, Resistor_SMD:R_0603_1608Metric, B.Cu at (129.8, 148.0)
- added R58: 1k, Resistor_SMD:R_0603_1608Metric, B.Cu at (129.6, 134.1)
- added R59: 1k, Resistor_SMD:R_0603_1608Metric, B.Cu at (140.8, 87.4)
- added R60: 0, Resistor_SMD:R_0603_1608Metric, F.Cu at (121.7, 93.2)
- added R61: 0, Resistor_SMD:R_0603_1608Metric, F.Cu at (172.7, 90.2)
- added R62: 0, Resistor_SMD:R_0603_1608Metric, F.Cu at (159.2, 90.2)
- added R63: 3.3K, Resistor_SMD:R_0603_1608Metric, F.Cu at (179.7, 23.8)
- added R64: 10k, Resistor_SMD:R_0603_1608Metric, F.Cu at (135.9, 60.6)
- added R65: XX, Resistor_SMD:R_0603_1608Metric, F.Cu at (118.9, 77.2)
- added R66: XX, Resistor_SMD:R_0603_1608Metric, F.Cu at (118.9, 79.7)
- added R67: 0, Resistor_SMD:R_0603_1608Metric, F.Cu at (203.5, 141.7)
- added R68: 0, Resistor_SMD:R_0603_1608Metric, F.Cu at (203.5, 144.2)
- added R69: 0, Resistor_SMD:R_0603_1608Metric, B.Cu at (104.6, 122.1)
- added R70: 0, Resistor_SMD:R_0603_1608Metric, B.Cu at (104.5, 123.6)
- added R71: 0, Resistor_SMD:R_0603_1608Metric, B.Cu at (100.5, 130.7)
- added R72: 0, Resistor_SMD:R_0603_1608Metric, F.Cu at (122.2, 122.7)
- added R73: 330, Resistor_SMD:R_0603_1608Metric, F.Cu at (119.1, 122.7)
- added R74: 330, Resistor_SMD:R_0603_1608Metric, F.Cu at (119.0, 124.6)
- added R75: 10k, Resistor_SMD:R_0603_1608Metric, B.Cu at (203.1, 63.8)
- added R76: 10k, Resistor_SMD:R_0603_1608Metric, B.Cu at (203.1, 66.3)
- added R77: 10k, Resistor_SMD:R_0603_1608Metric, F.Cu at (208.6, 97.5)
- added R78: 10k, Resistor_SMD:R_0603_1608Metric, F.Cu at (208.3, 114.3)
- added R79: 0.33, Resistor_THT:R_Axial_DIN0414_L11.9mm_D4.5mm_P15.24mm_Horizontal, F.Cu at (115.6, 40.4)
- added R80: 0.33, Resistor_THT:R_Axial_DIN0414_L11.9mm_D4.5mm_P15.24mm_Horizontal, F.Cu at (114.6, 59.1)
- added R81: 10k, Resistor_SMD:R_0603_1608Metric, B.Cu at (195.7, 61.7)
- added R82: 10k, Resistor_SMD:R_0603_1608Metric, B.Cu at (195.7, 64.2)
- added R83: 10k, Resistor_SMD:R_0603_1608Metric, B.Cu at (195.7, 66.7)
- added R84: 220, Resistor_SMD:R_0603_1608Metric, F.Cu at (108.4, 66.5)
- added R85: 220, Resistor_SMD:R_0603_1608Metric, F.Cu at (108.4, 69.0)
- added R86: 220, Resistor_SMD:R_0603_1608Metric, F.Cu at (108.4, 71.5)
- added R87: 220, Resistor_SMD:R_0603_1608Metric, F.Cu at (148.2, 88.8)
- added R88: 220, Resistor_SMD:R_0603_1608Metric, F.Cu at (151.6, 88.7)
- added R89: 220, Resistor_SMD:R_0603_1608Metric, F.Cu at (144.8, 88.7)
- added R90: 0, Resistor_SMD:R_0603_1608Metric, F.Cu at (185.4, 90.4)
- added R91: 330, Resistor_SMD:R_0603_1608Metric, F.Cu at (191.6, 90.4)
- added R92: 100k, Resistor_SMD:R_0603_1608Metric, B.Cu at (133.0, 128.4)
- added R93: 1k, Resistor_SMD:R_0603_1608Metric, B.Cu at (128.3, 142.2)
- added R94: 0, Resistor_SMD:R_0603_1608Metric, F.Cu at (121.9, 116.8)
- added R95: 330, Resistor_SMD:R_0603_1608Metric, F.Cu at (118.8, 116.8)
- added R96: 1k, Resistor_SMD:R_0603_1608Metric, B.Cu at (140.8, 89.9)
- added R97: 10k, Resistor_SMD:R_0603_1608Metric, B.Cu at (123.1, 71.0)
- added R98: 10k, Resistor_SMD:R_0603_1608Metric, B.Cu at (140.5, 64.7)
- added R99: 10k, Resistor_SMD:R_0603_1608Metric, B.Cu at (140.5, 67.2)
- added RV3: Vref_A, Potentiometer_SMD:Potentiometer_Bourns_3314S_Horizontal, B.Cu at (132.9, 78.5)
- added SW6: SW_User, Button_Switch_SMD:SW_Push_1P1T_NO_CK_KSC7xxJ, F.Cu at (149.0, 145.7)
- added SW7: SW_FORCE_ON, Button_Switch_SMD:SW_Push_1P1T_NO_CK_KSC7xxJ, F.Cu at (206.8, 56.4)
- added T1: TP, TestPoint:TestPoint_Pad_D1.0mm, B.Cu at (117.0, 139.8)
- added T10: TP, TestPoint:TestPoint_Pad_D1.0mm, F.Cu at (113.3, 112.0)
- added T11: TP, TestPoint:TestPoint_Pad_D1.0mm, F.Cu at (109.3, 98.2)
- added T12: TP, TestPoint:TestPoint_Pad_D1.0mm, F.Cu at (118.5, 96.4)
- added T13: TP, TestPoint:TestPoint_Pad_D1.0mm, F.Cu at (190.2, 135.2)
- added T14: TP, TestPoint:TestPoint_Pad_D1.0mm, F.Cu at (197.3, 136.7)
- added T15: TP, TestPoint:TestPoint_Pad_D1.0mm, F.Cu at (199.3, 135.3)
- added T16: TP, TestPoint:TestPoint_Pad_D1.0mm, F.Cu at (194.9, 135.3)
- added T17: TP, TestPoint:TestPoint_Pad_D1.0mm, F.Cu at (189.3, 128.3)
- added T18: TP, TestPoint:TestPoint_Pad_D1.0mm, F.Cu at (192.4, 135.3)
- added T19: TP, TestPoint:TestPoint_Pad_D1.0mm, F.Cu at (155.4, 136.1)
- added T2: TP, TestPoint:TestPoint_Pad_D1.0mm, F.Cu at (-11.5, 13.8)
- added T20: TP, TestPoint:TestPoint_Pad_D1.0mm, F.Cu at (144.3, 135.9)
- added T21: TP, TestPoint:TestPoint_Pad_D1.0mm, F.Cu at (144.3, 132.6)
- added T22: TP, TestPoint:TestPoint_Pad_D1.0mm, F.Cu at (142.9, 106.2)
- added T23: TP, TestPoint:TestPoint_Pad_D1.0mm, F.Cu at (142.8, 104.0)
- added T24: TP, TestPoint:TestPoint_Pad_D1.0mm, F.Cu at (143.0, 108.4)
- added T25: TP, TestPoint:TestPoint_Pad_D1.0mm, F.Cu at (152.8, 100.2)
- added T26: TP, TestPoint:TestPoint_Pad_D1.0mm, F.Cu at (151.9, 103.0)
- added T27: TP, TestPoint:TestPoint_Pad_D1.0mm, F.Cu at (146.2, 100.0)
- added T28: TP, TestPoint:TestPoint_Pad_D1.0mm, F.Cu at (139.8, 76.0)
- added T29: TP, TestPoint:TestPoint_Pad_D1.0mm, F.Cu at (142.8, 73.0)
- added T3: TP, TestPoint:TestPoint_Pad_D1.0mm, F.Cu at (139.8, 73.0)
- added T30: TP, TestPoint:TestPoint_Pad_D1.0mm, F.Cu at (144.8, 86.1)
- added T31: TP, TestPoint:TestPoint_Pad_D1.0mm, F.Cu at (151.6, 86.0)
- added T32: TP, TestPoint:TestPoint_Pad_D1.0mm, F.Cu at (148.2, 86.1)
- added T33: TP, TestPoint:TestPoint_Pad_D1.0mm, B.Cu at (111.8, 133.3)
- added T34: TP, TestPoint:TestPoint_Pad_D1.0mm, B.Cu at (111.8, 130.2)
- added T35: TP, TestPoint:TestPoint_Pad_D1.0mm, B.Cu at (249.2, 92.2)
- added T36: TP, TestPoint:TestPoint_Pad_D1.0mm, B.Cu at (249.2, 95.2)
- added T37: TP, TestPoint:TestPoint_Pad_D1.0mm, F.Cu at (203.0, 97.5)
- added T38: TP, TestPoint:TestPoint_Pad_D1.0mm, B.Cu at (128.9, 122.9)
- added T39: TP, TestPoint:TestPoint_Pad_D1.0mm, F.Cu at (148.9, 73.0)
- added T4: TP, TestPoint:TestPoint_Pad_D1.0mm, B.Cu at (109.3, 130.3)
- added T40: TP, TestPoint:TestPoint_Pad_D1.0mm, B.Cu at (112.1, 123.5)
- added T41: TP, TestPoint:TestPoint_Pad_D1.0mm, F.Cu at (105.6, 97.3)
- added T42: TP, TestPoint:TestPoint_Pad_D1.0mm, F.Cu at (146.3, 70.6)
- added T43: TP, TestPoint:TestPoint_Pad_D1.0mm, F.Cu at (157.8, 150.1)
- added T44: TP, TestPoint:TestPoint_Pad_D1.0mm, B.Cu at (249.2, 98.3)
- added T45: TP, TestPoint:TestPoint_Pad_D1.0mm, F.Cu at (160.6, 150.2)
- added T5: TP, TestPoint:TestPoint_Pad_D1.0mm, B.Cu at (113.8, 139.3)
- added T50: TP, TestPoint:TestPoint_Pad_D1.0mm, B.Cu at (249.2, 101.3)
- added T51: TP, TestPoint:TestPoint_Pad_D1.0mm, B.Cu at (249.2, 104.4)
- added T52: TP, TestPoint:TestPoint_Pad_D1.0mm, B.Cu at (118.8, 153.8)
- added T6: TP, TestPoint:TestPoint_Pad_D1.0mm, F.Cu at (-11.5, 16.9)
- added T7: TP, TestPoint:TestPoint_Pad_D1.0mm, B.Cu at (129.3, 119.8)
- added T8: TP, TestPoint:TestPoint_Pad_D1.0mm, B.Cu at (128.9, 125.1)
- added T9: TP, TestPoint:TestPoint_Pad_D1.0mm, F.Cu at (119.3, 107.9)
- added U16: LM317DCYG3, Package_TO_SOT_SMD:SOT-223-3_TabPin2, B.Cu at (184.6, 141.0)
- added U17: PCA9536D, Package_SO:SOIC-8_3.9x4.9mm_P1.27mm, B.Cu at (165.1, 130.7)
- added U18: 74LVC125, Package_SO:SSOP-14_5.3x6.2mm_P0.65mm, F.Cu at (191.8, 105.3)
- added U19: FT231XS, Package_SO:SSOP-20_3.9x8.7mm_P0.635mm, F.Cu at (195.5, 130.6)
- added U20: USBLC6-2P6, Package_TO_SOT_SMD:SOT-666, F.Cu at (198.6, 125.6)
- added U21: AS193-73, Package_TO_SOT_SMD:SOT-23-6, B.Cu at (119.5, 142.6)
- added U22: MCP4011, Package_SO:SOIC-8_3.9x4.9mm_P1.27mm, B.Cu at (112.7, 94.0)
- added U23: PC817, Package_SO:SOP-4_4.4x2.6mm_P1.27mm, F.Cu at (145.5, 94.6)
- added U24: PC817, Package_SO:SOP-4_4.4x2.6mm_P1.27mm, F.Cu at (152.2, 94.6)
- added U25: PC817, Package_SO:SOP-4_4.4x2.6mm_P1.27mm, F.Cu at (148.8, 94.6)
- added U26: USBLC6-2P6, Package_TO_SOT_SMD:SOT-666, B.Cu at (107.8, 124.0)
- added U27: LP2985-3.3, Package_TO_SOT_SMD:SOT-23-5, B.Cu at (101.1, 133.4)
- added U29: LM358DR, Package_SO:TSSOP-8_4.4x3mm_P0.65mm, B.Cu at (194.8, 71.5)
- AE1, C1, C12, C15, C16, C17, C18, C20, C4, C7, Q1, R13, R14, R30, R32, R36, R39, R42, R44, R48, R49, R5, R51, R6, R7, R8, R9, U11, U3: moved to B.Cu
- C10, C9: value 100pF -> 120pF; moved to B.Cu
- C11: value 100pF -> 100nF; moved to B.Cu
- C13: value 100nF -> 22uF; moved to B.Cu
- C14: value 1mF -> 100nF; moved to B.Cu
- C22, U15: moved to F.Cu
- D10, D12, D14, D7, D8, D9: footprint LED_THT:LED_D3.0mm -> LED_SMD:LED_0603_1608Metric
- D16: footprint Diode_SMD:D_0603_1608Metric -> Diode_SMD:D_SOD-323; moved to B.Cu
- D19: footprint Diode_THT:D_DO-41_SOD81_P7.62mm_Horizontal -> Diode_SMD:D_SOD-323; moved to B.Cu
- D2: value LED -> POS_ENABLE
- D3, D4, D5: footprint Diode_THT:D_DO-35_SOD27_P7.62mm_Horizontal -> Diode_SMD:D_SOD-323
- J10: value SPI_Programming -> 132415; footprint Connector_PinHeader_2.54mm:PinHeader_2x05_P2.54mm_Vertical -> Connector_Coaxial:SMA_Molex_73251-1153_EdgeMount_Horizontal; moved to B.Cu
- J11: value USR_BTN -> RST_BUTTON
- J12: value GND -> Analog_Pos; footprint Connector_PinHeader_2.54mm:PinHeader_1x01_P2.54mm_Vertical -> TerminalBlock_Phoenix:TerminalBlock_Phoenix_MPT-0,5-3-2.54_1x03_P2.54mm_Horizontal
- J16: footprint TerminalBlock_Phoenix:TerminalBlock_Phoenix_MPT-0,5-4-2.54_1x04_P2.54mm_Horizontal -> Connector_Phoenix_MSTB:PhoenixContact_MSTBA_2,5_4-G-5,08_1x04_P5.08mm_Horizontal
- J19: value USR_BTN -> USR_BTN_2
- J2: value RAW_data_Wind -> 132415; footprint Connector_PinHeader_2.54mm:PinHeader_1x01_P2.54mm_Vertical -> Connector_Coaxial:SMA_Molex_73251-1153_EdgeMount_Horizontal
- J3: value 132134 -> USB_C_Receptacle_USB2.0_16P; footprint Connector_Coaxial:SMA_Molex_73251-1153_EdgeMount_Horizontal -> Connector_USB:USB_C_Receptacle_GCT_USB4085
- J5: value Control -> USB_C_Receptacle_USB2.0_16P; footprint TerminalBlock_Phoenix:TerminalBlock_Phoenix_MPT-0,5-4-2.54_1x04_P2.54mm_Horizontal -> Connector_USB:USB_C_Receptacle_GCT_USB4085
- J6: footprint TerminalBlock_Phoenix:TerminalBlock_Phoenix_MKDS-1,5-2-5.08_1x02_P5.08mm_Horizontal -> Connector_Phoenix_MSTB:PhoenixContact_MSTBA_2,5_2-G-5,08_1x02_P5.08mm_Horizontal
- J7: footprint TerminalBlock_Phoenix:TerminalBlock_Phoenix_MKDS-3-2-5.08_1x02_P5.08mm_Horizontal -> Connector_Phoenix_MSTB:PhoenixContact_MSTBA_2,5_2-G-5,08_1x02_P5.08mm_Horizontal
- JP2: value Jumper -> Jumper_2_Open; footprint Connector_PinHeader_2.54mm:PinHeader_1x02_P2.54mm_Vertical -> Connector_PinHeader_1.27mm:PinHeader_1x02_P1.27mm_Vertical
- L1, L2, L3, L4: value L -> MPZ1608; moved to B.Cu
- Q3, Q8: footprint Package_TO_SOT_THT:TO-92_Inline -> Package_TO_SOT_SMD:SOT-23-3; moved to B.Cu
- R1: value 0 -> 330; moved to B.Cu
- R10, R47, R50: value 270 -> 330
- R17: value 0 -> 680k; moved to B.Cu
- R18: value 10k -> 0; moved to B.Cu
- R19: value 1k -> 270
- R2: value 1k -> 0; moved to B.Cu
- R3: value 2.2k -> 10k
- R33, R43: value 100k -> 1k; moved to B.Cu
- R52: value 270 -> 330; moved to B.Cu
- R53: value 1k -> 10k
- RV1: value R_Potentiometer -> Light_Reference; footprint Potentiometer_THT:Potentiometer_Bourns_3266Y_Vertical -> Potentiometer_SMD:Potentiometer_Bourns_3314S_Horizontal
- RV2: value R_Potentiometer -> Vref_B; footprint Potentiometer_THT:Potentiometer_Alps_RK163_Single_Horizontal -> Potentiometer_SMD:Potentiometer_Bourns_3314S_Horizontal; moved to B.Cu
- SW1, SW2, SW3, SW4, SW5: footprint Button_Switch_THT:SW_PUSH_6mm_H8mm -> Button_Switch_SMD:SW_Push_1P1T_NO_CK_KSC7xxJ
- U1: value LM358 -> LM358DR; footprint Package_SO:TSSOP-8_3x3mm_P0.65mm -> Package_SO:TSSOP-8_4.4x3mm_P0.65mm; moved to B.Cu
- U10: value L7805 -> ACS712xLCTR-05B; footprint Package_TO_SOT_THT:TO-220-3_Vertical -> Package_SO:SOIC-8_3.9x4.9mm_P1.27mm; moved to B.Cu
- U12: value LM317_TO-220 -> MC78L05_SOT89; footprint Package_TO_SOT_THT:TO-220-3_Vertical -> Package_TO_SOT_SMD:SOT-89-3; moved to B.Cu
- U13: footprint Package_SO:TSSOP-8_3x3mm_P0.65mm -> Package_SO:SO-8_5.3x6.2mm_P1.27mm; moved to B.Cu
- U2: value 74HC123 -> 74HC123D; footprint Package_SO:SSOP-16_4.4x5.2mm_P0.65mm -> Package_SO:SOIC-16W_5.3x10.2mm_P1.27mm
- U4: value AS193-73 -> XL1507; footprint Package_TO_SOT_SMD:SOT-23-6 -> Package_TO_SOT_SMD:TO-252-5_TabPin3; moved to B.Cu
- U5, U6, U7, U8, U9: footprint Package_DIP:DIP-4_W7.62mm -> Package_SO:SOP-4_4.4x2.6mm_P1.27mm
- Y1: footprint Crystal:Crystal_HC49-4H_Vertical -> Crystal:Crystal_SMD_HC49-SD
- Y2: footprint Crystal:Crystal_AT310_D3.0mm_L10.0mm_Horizontal -> Crystal:Crystal_SMD_3215-2Pin_3.2x1.5mm; moved to B.Cu
- moved R2 197.3 mm to (2.28, 17.4), turned to 180 degrees
- moved C12 133.3 mm to (39.1, 1.96), turned to 180 degrees
- moved C13 133.3 mm to (39.1, 4.47), turned to 180 degrees
- moved H4 123.9 mm to (201.2, 25.1)
- moved J16 121.3 mm to (108.2, 42.7), turned to -90 degrees
- moved J10 118.8 mm to (108.6, 155.0), turned to 90 degrees
- moved H1 117.5 mm to (98.7, 23.5)
- moved L4 114.0 mm to (207.2, 90.2), turned to -90 degrees
- moved C14 104.2 mm to (187.9, 75.9)
- moved U12 101.9 mm to (189.1, 79.8)
- moved C15 100.8 mm to (197.9, 126.2), turned to -90 degrees
- moved J12 98.6 mm to (119.1, 24.9), turned to 180 degrees
- moved L3 96.7 mm to (197.9, 130.2), turned to -90 degrees
- moved JP8 96.0 mm to (169.9, 24.1), turned to -90 degrees
- moved U10 93.6 mm to (189.8, 88.8), turned to 180 degrees
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Connections:
- C1 pad 1: +5V -> +5V_Security
- C1 pad 2: GND -> GND_Security
- C10 pad 1: Net-(AE1-A) -> Net-(U21-J2)
- C10 pad 2: Net-(U4-RF1) -> Net-(AE1-A)
- C11 pad 1: Net-(J3-In) -> GND
- C11 pad 2: Net-(U4-RF2) -> +5V
- C13 pad 1: Net-(JP3-A) -> Net-(D16-K)
- C14 pad 1: Net-(JP3-A) -> Net-(D16-K)
- C17 pad 1: Net-(JP5-A) -> +3.3V
- C20 pad 1: GND -> +5V
- C20 pad 2: +5V -> GND
- C3 pad 1: +5V -> +5V_Security
- C3 pad 2: GND -> GND_Security
- C4 pad 2: GND -> GND_Security
- C9 pad 1: Net-(U4-RFC) -> Net-(U21-J1)
- D19 pad 2: Net-(D19-A) -> /Power_Supply/Vcapa
- D3 pad 1: /Motors/ENABLE -> /Motors/ENABLED
- D3 pad 2: Net-(D3-A) -> /MCU/PD3-D3-(INT1)~
- D4 pad 2: Net-(D4-A) -> /MCU/PD5-D5~
- D5 pad 2: Net-(D5-A) -> /MCU/PD4-D4
- D7 pad 2: /Motors/IN_B -> /MCU/PD4-D4
- D8 pad 2: /Motors/IN_A -> /MCU/PD5-D5~
- J1 pad 2: GND -> GND_Security
- J10 pad 1: /MCU/MOSI -> Net-(J10-In)
- J10 pad 2: +3.3V -> GND_GNSS
- J11 pad 1: /RST -> GND
- J11 pad 2: GND -> /MCU/~{RESET}/PC6
- J16 pad 1: /MCU/PB0 -> Net-(IC1-OUT1A)
- J16 pad 2: /MCU/PB1-D9~ -> Net-(IC1-OUT2A)
- J16 pad 3: /MCU/PB2-D10~ -> Net-(IC1-OUT1B)
- J16 pad 4: GND -> Net-(IC1-OUT2B)
- J19 pad 1: /UserActions/Button -> +5V
- J19 pad 2: +5V -> /MCU/PC2-A2
- J4 pad 1: Net-(D3-A) -> /MCU/PD3-D3-(INT1)~
- J4 pad 2: Net-(D4-A) -> /MCU/PD5-D5~
- J4 pad 3: Net-(D5-A) -> /MCU/PD4-D4
- JP2 pad 1: /+24V -> Net-(JP2-A)
- JP2 pad 2: Net-(D16-A) -> /MCU/PB0
- JP8 pad 1: Net-(JP8-A) -> Net-(J23-Pin_1)
- JP8 pad 2: Net-(JP8-B) -> /Motors/ENABLED
- L4 pad 2: GND_GNSS -> GND
- Q1 pad 1: /GNSS/~{INTERNAL_ANTENNA} -> /GNSS/~{ANTENNA_DETECT}
- Q1 pad 2: GND_GNSS -> Net-(Q1-S)
- Q1 pad 3: Net-(Q1-D) -> GND_GNSS
- R1 pad 1: /GNSS/~{INTERNAL_ANTENNA} -> Net-(D21-K)
- R1 pad 2: /MCU/PD7-D7 -> GND
- R10 pad 2: GND -> GND_Security
- R11 pad 1: /GNSS/RX -> /GNSS_TX
- R12 pad 1: /GNSS/TX -> /GNSS_RX
- R14 pad 1: Net-(U3-RXD/SPI_MOSI) -> GND_GNSS
- R14 pad 2: GND_GNSS -> Net-(U3-RXD/SPI_MOSI)
- R17 pad 1: Net-(U3-TIMEPULSE) -> /GNSS/~{ANTENNA_DETECT}
- R17 pad 2: /TIMEPULSE -> /GNSS/VCC_RF
- R18 pad 1: GND_GNSS -> Net-(U13-SQW/OUT)
- R18 pad 2: /GNSS/~{INTERNAL_ANTENNA} -> Net-(R18-Pad2)
- R19 pad 1: Net-(Q1-D) -> Net-(D25-K)
- R19 pad 2: +3.3V_GNSS -> GND
- R2 pad 1: /V_{A_{2}} -> /WIND_INTERRUPT
- R2 pad 2: /UserActions/Button -> /Power_Supply/WakeUp_Handler/WIND_INTERRUPT
- R20 pad 2: Net-(SW1A-B) -> Net-(J28-Pin_2)
- R23 pad 1: /Motors/ENABLE -> Net-(J23-Pin_2)
- R3 pad 1: /V_{A_{2}} -> /MCU/PC2-A2
- R3 pad 2: /TIMEPULSE -> GND
- R4 pad 1: +5V -> +5V_Security
- R46 pad 2: /RST -> /MCU/~{RESET}/PC6
- R48 pad 2: Net-(U12-ADJ) -> Net-(U16-ADJ)
- R49 pad 1: Net-(U12-ADJ) -> Net-(U16-ADJ)
- R5 pad 1: +5V -> +5V_Security
- R52 pad 2: Net-(JP8-B) -> Net-(R18-Pad2)
- R53 pad 1: /UserActions/Button -> /MCU/PC1-A1
- R8 pad 2: /MCU/PD2-D2-(INT0) -> Net-(R104-Pad1)
- R9 pad 1: GND -> GND_Security
- R9 pad 2: /MCU/PD2-D2-(INT0) -> Net-(R104-Pad1)
- RV1 pad 1: +5V -> GND_Security
- RV1 pad 2: Net-(U1A--) -> Net-(U29A--)
- RV1 pad 3: GND -> +5V_Security
- RV2 pad 2: /MCU/PC1-A1 -> /Stepper/Vref_B
- SW1 pad 1: /Motors/ENABLE -> Net-(J28-Pin_2)
- SW1 pad 2: Net-(SW1A-B) -> /Motors/ENABLED
- SW4 pad 2: /RST -> /MCU/~{RESET}/PC6
- SW5 pad 2: /UserActions/Button -> /MCU/PC1-A1
- U1 pad 1: /MCU/PD2-D2-(INT0) -> Net-(R104-Pad1)
- U1 pad 4: GND -> GND_Security
- U1 pad 8: +5V -> +5V_Security
- U10 pad 1: Net-(D16-K) -> +24V
- U10 pad 2: GND -> +24V
- U10 pad 3: Net-(JP3-A) -> Net-(D16-A)
- U11 pad 2: Net-(JP5-A) -> +3.3V
- U12 pad 1: Net-(U12-ADJ) -> Net-(U12-OUT)
- U12 pad 2: /Power_Supply/Vcapa -> GND
- U12 pad 3: +5V -> Net-(D16-K)
- U13 pad 7: Net-(JP8-A) -> Net-(U13-SQW/OUT)
- U14 pad 3: /MCU/PD6-D6~ -> /MCU/A6
- U15 pad 1: /MCU/PD3-D3-(INT1)~ -> Net-(JP24-A)
- U15 pad 10: /MCU/PD6-D6~ -> Net-(JP27-A)
- U15 pad 11: /MCU/PD7-D7 -> Net-(JP26-A)
- U15 pad 12: /MCU/PB0 -> Net-(JP2-A)
- U15 pad 13: /MCU/PB1-D9~ -> Net-(JP9-A)
- U15 pad 14: /MCU/PB2-D10~ -> Net-(JP10-A)
- U15 pad 15: /MCU/MOSI -> Net-(JP11-A)
- U15 pad 16: /MCU/MISO -> Net-(JP12-A)
- U15 pad 17: /MCU/CLK -> Net-(JP13-A)
- U15 pad 19: unconnected-(U15-ADC6-Pad19) -> /MCU/A6
- U15 pad 2: /MCU/PD4-D4 -> Net-(JP25-A)
- U15 pad 22: unconnected-(U15-ADC7-Pad22) -> /MCU/A7
- U15 pad 23: /MCU/PC0-A0 -> Net-(JP14-A)
- U15 pad 24: /MCU/PC1-A1 -> Net-(JP15-A)
- U15 pad 25: /V_{A_{2}} -> Net-(JP16-A)
- U15 pad 26: /MCU/PC3-A3 -> Net-(JP17-A)
- U15 pad 27: /Anemometer/SDA -> Net-(JP18-A)
- U15 pad 28: /Anemometer/SCL -> Net-(JP19-A)
- U15 pad 29: /RST -> Net-(JP20-A)
- U15 pad 30: /GNSS/RX -> Net-(JP21-A)
- U15 pad 31: /GNSS/TX -> Net-(JP22-A)
- U15 pad 32: /MCU/PD2-D2-(INT0) -> Net-(JP23-A)
- U15 pad 9: /MCU/PD5-D5~ -> Net-(JP28-A)
- U2 pad 1: unconnected-(U2A-A-Pad1) -> /SIMULATE_WIND
- U2 pad 16: +5V -> +5V_Security
- U2 pad 3: GND -> GND_Security
- U2 pad 8: GND -> GND_Security
- U3 pad 1: unconnected-(U3-~{SAFEBOOT}-Pad1) -> Net-(U3-~{SAFEBOOT})
- U3 pad 18: unconnected-(U3-SDA/~{SPI_CS}-Pad18) -> Net-(U3-SDA/~{SPI_CS})
- U3 pad 19: unconnected-(U3-SCL/SPI_CLK-Pad19) -> Net-(U3-SCL/SPI_CLK)
- U3 pad 2: unconnected-(U3-D_SEL-Pad2) -> Net-(U3-D_SEL)
- U3 pad 23: +3.3V_GNSS -> Net-(Q10-D)
- U3 pad 4: unconnected-(U3-EXTINT-Pad4) -> Net-(U3-EXTINT)
- U3 pad 5: unconnected-(U3-USB_DM-Pad5) -> /GNSS/D-
- U3 pad 6: unconnected-(U3-USB_DP-Pad6) -> /GNSS/D+
- U3 pad 7: unconnected-(U3-VDD_USB-Pad7) -> /GNSS/VCC_USB
- U3 pad 9: unconnected-(U3-VCC_RF-Pad9) -> /GNSS/VCC_RF
- U4 pad 1: Net-(U4-RF1) -> Net-(D16-K)
- U4 pad 2: GND_GNSS -> Net-(D23-K)
- U4 pad 3: Net-(U4-RF2) -> GND
- U4 pad 4: /GNSS/~{INTERNAL_ANTENNA} -> Net-(U4-Feedback)
- U4 pad 5: Net-(U4-RFC) -> /Power_Supply/WakeUp_Handler/PS_CTRL
Routing:
- net +5V: track 0.00 -> 172.8 mm, vias 0 -> 10
- net +5V_Security: track 0.00 -> 65.8 mm, vias 0 -> 4
- net +3.3V_GNSS: track 0.00 -> 53.1 mm, vias 0 -> 5
- net /GNSS/VCC_USB: track 0.00 -> 52.1 mm, vias 0 -> 4
- net Net-(IC1-OUT2A): track 0.00 -> 50.8 mm
- net /Anemometer/SCL: track 0.00 -> 49.8 mm, vias 0 -> 3
- net /Anemometer/SDA: track 0.00 -> 48.4 mm, vias 0 -> 2
- net +3.3V: track 0.00 -> 46.9 mm, vias 0 -> 3
- net Net-(R104-Pad1): track 0.00 -> 46.8 mm, vias 0 -> 1
- net /GNSS_ENABLED: track 0.00 -> 46.7 mm, vias 0 -> 1
- net Net-(Q1-S): track 0.00 -> 44.8 mm, vias 0 -> 3
- net /GNSS/~{ANTENNA_DETECT}: track 0.00 -> 43.3 mm, vias 0 -> 2
- net Net-(Q10-G): track 0.00 -> 41.7 mm
- net Net-(U3-TXD/SPI_MISO): track 0.00 -> 40.9 mm, vias 0 -> 3
- net /GNSS/VCC_RF: track 0.00 -> 37.7 mm, vias 0 -> 2
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- added copper zone on B.Cu, net GND
- added copper zone on F.Cu, net GND
- added copper zone on B.Cu, net GND_GNSS
- added copper zone on F.Cu, net GND_GNSS
- added copper zone on B.Cu, net GND_Security
- added copper zone on F.Cu, net GND_Security
Other:
- board outline added: 115.8 x 141.2 mm
- board text added: "+24V.GND - Stepper"
- board text added: "+3.3V_GNSS"
- board text added: "+5V.SCL.SDA.GND"
- board text added: "+5V_ON"
- board text added: "+5V_SECURITY"
- board text added: "A1_A2_B1_B2"
- board text added: "ALERT"
- board text added: "ANEMO"
- board text added: "ANEMO.IN"
- board text added: "ANEMO.OUT"
- board text added: "BTN_1"
- board text added: "BTN_2"
- board text added: "CLK"
- board text added: "DIR.EN.PULSE"
- board text added: "EN.In_A.In_B"
- board text added: "END_STP_1"
- board text added: "END_STP_2"
- board text added: "EXT_ANT"
- board text added: "GND.+24V"
- board text added: "GNSS_BATT"
- board text added: "GNSS_POS"
- board text added: "GNSS_USB"
- board text added: "LDR"
- board text added: "MISO"
- board text added: "MOSI"
- board text added: "ON_B"
- board text added: "ORIGIN"
- board text added: "On/OFF"
- board text added: "PCB3D_TL_CMS"
- board text added: "PROJET CREPP Tracker solaire 2023-2024 - V2"
- board text added: "RESET"
- board text added: "RTC"
- board text added: "SCL"
- board text added: "SDA"
- board text added: "SELF_TEST"
- board text removed: "16MHz"
