File: Hardware/V2_CMS/Tracker.kicad_sch (KiCad schematic)
At the start: 7 parts

Commit message: update of directory
Parts:
- removed R1: 0, Resistor_SMD:R_0603_1608Metric, symbol Device:R
- removed R2: 1k, Resistor_SMD:R_0603_1608Metric, symbol Device:R
- removed R3: 2.2k, Resistor_SMD:R_0603_1608Metric, symbol Device:R
- added H5, H6, H7, H8: Probe_GND, Holes:Hole_1mm_Scope, symbol Mechanical:MountingHole_Pad
Connections:
- net GND: now also H5.1, H6.1, H7.1, H8.1
Other:
- added sheet IO_Extender (Modules/IO_Extender.kicad_sch)
- added sheet SD_Reader (Modules/SD_Reader.kicad_sch)
- sheet GNSS ports: added GNSS_ENABLED, GNSS_RX, GNSS_TX; removed TIMEPULSE, {UART}, ~{INTERNAL_ANTENNA}
- sheet MCU ports: added A6, A7; removed none
- sheet Motors ports: added Analog_Position, M_ENABLED; removed Analog_position, M_ENABLE
- sheet Power_Supply ports: added +5V_SECURITY, GND_Power, GND_Security, WIND_INTERRUPT; removed none
- sheet Programming ports: added +5V, {UART}; removed AVR_ISP_RST, AVR_SPI_+5V, {SPI}
- sheet Stepper ports: added +24V, +5V, Stepper_CW/~{CCW}, Stepper_Enable, Stepper_Pulse, ~{Stepper_Origine}; removed Dir, Enable, Pulse
- sheet UserActions ports: added USR_BTN_1, USR_BTN_2; removed Button, POT
- sheet WIND ports: added Simulation, U/~{D}, Wind_interrupt_MCU, Wind_interrupt_Power, ~{CS}; removed Wind_interrupt
- note removed: "TIMEPULSE == 0 && Button == Released : V_{A2} = 0V TIMEPULSE == 0 && Button == Pressed : V_{A2} = Vcc TIMEPULSE == 1 && Button == Released : V_{A2} = 5*({R31:value}/({R31:value})) TIMEPULSE == 1 && Button == Pressed : V_{A2} = 5*({R31:value}/({R31:value}))"
- moved on the sheet: H1, H2, H3, H4
