File: Hardware/V2_CMS/UserActions.kicad_sch (KiCad schematic)
At the start: 4 parts, among them J19 USR_BTN, SW5 SW_User

Commit message: update of directory
Parts:
- removed J19: USR_BTN, TerminalBlock_Phoenix:TerminalBlock_Phoenix_MPT-0,5-2-2.54_1x02_P2.54mm_Horizontal, symbol Connector:Conn_01x02_Pin
- removed RV2: R_Potentiometer, Potentiometer_THT:Potentiometer_Alps_RK163_Single_Horizontal, symbol Device:R_Potentiometer
- added J19: USR_BTN_2, TerminalBlock_Phoenix:TerminalBlock_Phoenix_MPT-0,5-2-2.54_1x02_P2.54mm_Horizontal, symbol Connector:Screw_Terminal_01x02
- added J21: USR_BTN_1, TerminalBlock_Phoenix:TerminalBlock_Phoenix_MPT-0,5-2-2.54_1x02_P2.54mm_Horizontal, symbol Connector:Screw_Terminal_01x02
- added R3: 10k, Resistor_SMD:R_0603_1608Metric, symbol PCM_SL_Devices:Resistor_0.5W
- added SW6: SW_User, Button_Switch_SMD:SW_Push_1P1T_NO_CK_KSC7xxJ, symbol Switch:SW_DPST_x2
- R53: value 1k -> 10k
- SW5: footprint Button_Switch_THT:SW_PUSH_6mm_H8mm -> Button_Switch_SMD:SW_Push_1P1T_NO_CK_KSC7xxJ
Connections:
- net GND: now also R3.2
- net VCC: now also J19.1 (Pin_1), J21.1 (Pin_1), SW6.1 (A)
- net Button renamed USR_BTN_1
- net USR_BTN_1: now also J21.2 (Pin_2)
- new net USR_BTN_2: J19.2 (Pin_2), R3.1, SW6.2 (B)
