File: Hardware/V2_CMS/Modules/Motor_Control.kicad_sch (KiCad schematic)
At the start: 71 parts, among them J4 PinHeader_Control, J5 Control, J6 +24V, J7 Motor, Q2 IRF4905, Q3 2N7000, Q4 IRF4905, Q5 IRF520, Q6 IRF4905, Q7 IRF520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

Commit message: update of directory
Parts:
- removed F1: Fuse, Fuse:Fuseholder_Cylinder-5x20mm_Schurter_0031_8201_Horizontal_Open, symbol Device:Fuse
- removed H10, H11, H12, H9: Probe_GND, Holes:Hole_1mm_Scope, symbol Mechanical:MountingHole_Pad
- removed H5, H6, H7, H8: MountingHole, MountingHole:MountingHole_3mm, symbol Mechanical:MountingHole
- removed J5: Control, TerminalBlock_Phoenix:TerminalBlock_Phoenix_MPT-0,5-4-2.54_1x04_P2.54mm_Horizontal, symbol Connector:Screw_Terminal_01x04
- added HS5: Heatsink, HeatSink:HeastSink_MOSFET_15mm_10mm_20mm, symbol Mechanical:Heatsink
- added J12: Analog_Pos, TerminalBlock_Phoenix:TerminalBlock_Phoenix_MPT-0,5-3-2.54_1x03_P2.54mm_Horizontal, symbol Connector:Screw_Terminal_01x03
- added J23, J25: END_STOP_1, TerminalBlock_Phoenix:TerminalBlock_Phoenix_MPT-0,5-2-2.54_1x02_P2.54mm_Horizontal, symbol Connector:Screw_Terminal_01x02
- added J27: EN_LED, TerminalBlock_Phoenix:TerminalBlock_Phoenix_MPT-0,5-2-2.54_1x02_P2.54mm_Horizontal, symbol Connector:Screw_Terminal_01x02
- added J28: SW_EN, TerminalBlock_Phoenix:TerminalBlock_Phoenix_MPT-0,5-2-2.54_1x02_P2.54mm_Horizontal, symbol Connector:Screw_Terminal_01x02
- added J29: EXT_SW_A, TerminalBlock_Phoenix:TerminalBlock_Phoenix_MPT-0,5-2-2.54_1x02_P2.54mm_Horizontal, symbol Connector:Screw_Terminal_01x02
- added J30: EXT_SW_B, TerminalBlock_Phoenix:TerminalBlock_Phoenix_MPT-0,5-2-2.54_1x02_P2.54mm_Horizontal, symbol Connector:Screw_Terminal_01x02
- added J33: Fuse, Connector_Phoenix_MSTB:PhoenixContact_MSTBA_2,5_2-G-5,08_1x02_P5.08mm_Horizontal, symbol Connector:Screw_Terminal_01x02
- added JP29, JP8: Jumper, Connector_PinHeader_2.54mm:PinHeader_1x02_P2.54mm_Vertical, symbol Jumper:Jumper_2_Bridged
- added R102: 0, Resistor_SMD:R_0603_1608Metric, symbol PCM_SL_Devices:Resistor_0.5W
- added R59, R96: 1k, Resistor_SMD:R_0603_1608Metric, symbol PCM_SL_Devices:Resistor_0.5W
- added R63: 3.3K, Resistor_SMD:R_0603_1608Metric, symbol PCM_SL_Devices:Resistor_0.5W
- D10, D12, D14, D7, D8, D9: footprint LED_THT:LED_D3.0mm -> LED_SMD:LED_0603_1608Metric
- D3, D4, D5: footprint Diode_THT:D_DO-35_SOD27_P7.62mm_Horizontal -> Diode_SMD:D_SOD-323
- J6: footprint TerminalBlock_Phoenix:TerminalBlock_Phoenix_MKDS-1,5-2-5.08_1x02_P5.08mm_Horizontal -> Connector_Phoenix_MSTB:PhoenixContact_MSTBA_2,5_2-G-5,08_1x02_P5.08mm_Horizontal
- J7: footprint TerminalBlock_Phoenix:TerminalBlock_Phoenix_MKDS-3-2-5.08_1x02_P5.08mm_Horizontal -> Connector_Phoenix_MSTB:PhoenixContact_MSTBA_2,5_2-G-5,08_1x02_P5.08mm_Horizontal
- Q3, Q8: footprint Package_TO_SOT_THT:TO-92_Inline -> Package_TO_SOT_SMD:SOT-23-3
- R33, R43: value 100k -> 1k
- SW1, SW2, SW3: footprint Button_Switch_THT:SW_PUSH_6mm_H8mm -> Button_Switch_SMD:SW_Push_1P1T_NO_CK_KSC7xxJ
- U5, U6, U7, U8, U9: footprint Package_DIP:DIP-4_W7.62mm -> Package_SO:SOP-4_4.4x2.6mm_P1.27mm
Connections:
- net +VCC_Motor: now also J12.3 (Pin_3), J27.1 (Pin_1)
- net GND: now also J12.1 (Pin_1), R63.1, R96.1
- net IN_A: now also J29.2 (Pin_2); no longer D8.2 (A)
- net IN_B: now also J30.1 (Pin_1); no longer D7.2 (A)
- net at R20.2: now also SW1.1 (A), J28.2 (Pin_2); no longer SW1.2 (B)
- net M_ENABLED: now reaches D3.2 (A), J4.1 (Pin_1)
- net M_IN_A: now reaches D4.2 (A), J4.2 (Pin_2)
- net M_IN_A: now also D8.2 (A)
- net M_IN_B: now reaches D5.2 (A), J4.3 (Pin_3)
- net M_IN_B: now also D7.2 (A)
- net at D9.2 (A), Q2.3 (S), R27.2: now also J33.1 (Pin_1)
- net at D6.1 (K), R20.1: now also J33.2 (Pin_2)
- net at R21.2, SW2.2 (B): now also J30.2 (Pin_2)
- net at R24.2, SW3.2 (B): now also J29.1 (Pin_1)
- removed net ENABLE: D3.1 (K), R23.1, SW1.1 (A)
- new net: J23.2 (Pin_2), JP29.1 (A), R23.1
- new net: J23.1 (Pin_1), J25.2 (Pin_2), JP29.2 (B), JP8.1 (A)
- new net: R102.1, R59.2, R96.2
- new net: J12.2 (Pin_2), R59.1
- new net: J27.2 (Pin_2), R63.2
- new net Analog_Position: R102.2
- new net ENABLED: D3.1 (K), J25.1 (Pin_1), J28.1 (Pin_1), JP8.2 (B), SW1.2 (B)
Other:
- moved on the sheet: D10, D6, D7, D8, D9, J6, Q2, R20, R22, R23, R25, R26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
