File: Hardware/V2_CMS/Modules/RTC.kicad_sch (KiCad schematic)
At the start: 6 parts, among them U13 DS1307+, Y2 32kHz

Commit message: update of directory
Parts:
- removed JP8: Jumper, Connector_PinHeader_2.54mm:PinHeader_1x02_P2.54mm_Vertical, symbol Jumper:Jumper_2_Bridged
- added R18: 0, Resistor_SMD:R_0603_1608Metric, symbol Device:R
- added T19: TP, TestPoint:TestPoint_Pad_D1.0mm, symbol Connector:TestPoint
- R52: value 270 -> 330
- U13: footprint Package_SO:TSSOP-8_3x3mm_P0.65mm -> Package_SO:SO-8_5.3x6.2mm_P1.27mm
- Y2: footprint Crystal:Crystal_AT310_D3.0mm_L10.0mm_Horizontal -> Crystal:Crystal_SMD_3215-2Pin_3.2x1.5mm
Connections:
- net +5V: now also C20.1; no longer C20.2
- net GND: now also C20.2; no longer C20.1
- net at U13.7 (SQW/OUT): now also R18.1, T19.1
- net at R52.2: now also R18.2
Other:
- moved on the sheet: C20
Changed lines of the file:
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@@
 	)
 	(junction
-		(at 90.17 52.07)
+		(at 113.03 66.04)
+		(diameter 0)
+		(color 0 0 0 0)
+	)
+	(junction
+		(at 82.55 43.18)
 		(diameter 0)
 		(color 0 0 0 0)
@@
 	(wire
 		(pts
+			(xy 82.55 43.18) (xy 93.98 43.18)
+		)
+		(stroke
+			(width 0)
+			(type default)
+		)
+	)
+	(wire
+		(pts
+			(xy 93.98 43.18) (xy 93.98 55.88)
+		)
+		(stroke
+			(width 0)
+			(type default)
+		)
+	)
+	(wire
+		(pts
 			(xy 96.52 76.2) (xy 96.52 80.01)
 		)
@@
 	(wire
 		(pts
-			(xy 127 66.04) (xy 129.54 66.04)
+			(xy 113.03 66.04) (xy 116.84 66.04)
 		)
 		(stroke
@@
 	(wire
 		(pts
-			(xy 90.17 50.8) (xy 90.17 52.07)
-		)
-		(stroke
-			(width 0)
-			(type default)
-		)
-	)
-	(wire
-		(pts
 			(xy 72.39 76.2) (xy 72.39 68.58)
 		)
@@
 	(wire
 		(pts
-			(xy 90.17 36.83) (xy 90.17 43.18)
+			(xy 78.74 43.18) (xy 82.55 43.18)
+		)
+		(stroke
+			(width 0)
+			(type default)
+		)
+	)
+	(wire
+		(pts
+			(xy 82.55 52.07) (xy 82.55 54.61)
+		)
+		(stroke
+			(width 0)
+			(type default)
+		)
+	)
+	(wire
+		(pts
+			(xy 113.03 66.04) (xy 113.03 69.85)
+		)
+		(stroke
+			(width 0)
+			(type default)
+		)
+	)
+	(wire
+		(pts
+			(xy 124.46 66.04) (xy 129.54 66.04)
 		)
 		(stroke
@@
 	(wire
 		(pts
-			(xy 93.98 52.07) (xy 93.98 55.88)
-		)
-		(stroke
-			(width 0)
-			(type default)
-		)
-	)
-	(wire
-		(pts
 			(xy 129.54 46.99) (xy 129.54 50.8)
 		)
@@
 	(wire
 		(pts
-			(xy 109.22 66.04) (xy 116.84 66.04)
+			(xy 82.55 43.18) (xy 82.55 44.45)
+		)
+		(stroke
+			(width 0)
+			(type default)
+		)
+	)
+	(wire
+		(pts
+			(xy 109.22 66.04) (xy 113.03 66.04)
 		)
 		(stroke
@@
 		(pts
 			(xy 81.28 76.2) (xy 82.55 76.2)
-		)
-		(stroke
-			(width 0)
-			(type default)
-		)
-	)
-	(wire
-		(pts
-			(xy 82.55 52.07) (xy 90.17 52.07)
-		)
-		(stroke
-			(width 0)
-			(type default)
-		)
-	)
-	(wire
-		(pts
-			(xy 90.17 52.07) (xy 93.98 52.07)
 		)
 		(stroke
@@
 	)
 	(label "GND"
-		(at 90.17 36.83 0)
-		(fields_autoplaced yes)
-		(effects
-			(font
-				(size 1.27 1.27)
-			)
-			(justify left bottom)
+		(at 82.55 54.61 180)
+		(fields_autoplaced yes)
+		(effects
+			(font
+				(size 1.27 1.27)
+			)
+			(justify right bottom)
 		)
 	)
@@
 	(hierarchical_label "+5V"
 		(shape input)
-		(at 82.55 52.07 180)
+		(at 78.74 43.18 180)
 		(fields_autoplaced yes)
 		(effects
@@
 	)
 	(symbol
-		(lib_id "Jumper:Jumper_2_Bridged")
-		(at 121.92 66.04 0)
+		(lib_id "Device:R")
+		(at 120.65 66.04 90)
 		(unit 1)
-		(exclude_from_sim yes)
+		(exclude_from_sim no)
 		(in_bom yes)
 		(on_board yes)
 		(dnp no)
-		(property "Reference" "JP8"
-			(at 126.238 64.77 0)
-			(effects
-				(font
-					(size 1.27 1.27)
-				)
-			)
-		)
-		(property "Value" "Jumper"
-			(at 121.92 63.5 0)
-			(effects
-				(font
-					(size 1.27 1.27)
-				)
-				(hide yes)
-			)
-		)
-		(property "Footprint" "Connector_PinHeader_2.54mm:PinHeader_1x02_P2.54mm_Vertical"
-			(at 121.92 66.04 0)
+		(fields_autoplaced yes)
+		(property "Reference" "R18"
+			(at 120.65 59.69 90)
+			(effects
+				(font
+					(size 1.27 1.27)
+				)
+			)
+		)
+		(property "Value" "0"
+			(at 120.65 62.23 90)
+			(effects
+				(font
+					(size 1.27 1.27)
+				)
+			)
+		)
+		(property "Footprint" "Resistor_SMD:R_0603_1608Metric"
+			(at 120.65 67.818 90)
 			(effects
 				(font
@@
 		)
 		(property "Datasheet" "~"
-			(at 121.92 66.04 0)
-			(effects
-				(font
-					(size 1.27 1.27)
-				)
-				(hide yes)
-			)
-		)
-		(property "Description" "Jumper, 2-pole, closed/bridged"
-			(at 121.92 66.04 0)
+			(at 120.65 66.04 0)
+			(effects
+				(font
+					(size 1.27 1.27)
+				)
+				(hide yes)
+			)
+		)
+		(property "Description" ""
+			(at 120.65 66.04 0)
 			(effects
 				(font
@@
 			(project "Tracker"
 				(path "/60c5e70b-bc37-4402-aa86-9378cecb8f85/5d9555c7-4fd3-4187-a03c-c3d0cf6806ca"
-					(reference "JP8")
+					(reference "R18")
 					(unit 1)
 				)
@@
 	(symbol
 		(lib_id "Device:C")
-		(at 90.17 46.99 0)
+		(at 82.55 48.26 0)
 		(unit 1)
 		(exclude_from_sim no)
@@
 		(dnp no)
 		(property "Reference" "C20"
-			(at 88.138 53.086 90)
+			(at 83.82 50.8 0)
 			(effects
 				(font
@@
 		)
 		(property "Value" "100nF"
-			(at 88.138 44.704 90)
+			(at 84.074 45.466 0)
 			(effects
 				(font
@@
 		)
 		(property "Footprint" "Capacitor_SMD:C_0603_1608Metric"
-			(at 91.1352 50.8 0)
+			(at 83.5152 52.07 0)
 			(effects
 				(font
@@
 		)
 		(property "Datasheet" "~"
-			(at 90.17 46.99 0)
+			(at 82.55 48.26 0)
 			(effects
 				(font
@@
 		)
 		(property "Description" ""
-			(at 90.17 46.99 0)
+			(at 82.55 48.26 0)
 			(effects
 				(font
@@
 				(path "/60c5e70b-bc37-4402-aa86-9378cecb8f85/5d9555c7-4fd3-4187-a03c-c3d0cf6806ca"
 					(reference "C20")
+					(unit 1)
+				)
+			)
+		)
+	)
+	(symbol
+		(lib_id "Connector:TestPoint")
+		(at 113.03 69.85 180)
+		(unit 1)
+		(exclude_from_sim no)
+		(in_bom yes)
+		(on_board yes)
+		(dnp no)
+		(property "Reference" "T19"
+			(at 113.03 77.216 90)
+			(effects
+				(font
+					(size 1.27 1.27)
+				)
+			)
+		)
+		(property "Value" "TP"
+			(at 110.49 73.152 90)
+			(effects
+				(font
+					(size 1.27 1.27)
+				)
+				(hide yes)
+			)
+		)
+		(property "Footprint" "TestPoint:TestPoint_Pad_D1.0mm"
+			(at 107.95 69.85 0)
+			(effects
+				(font
+					(size 1.27 1.27)
+				)
+				(hide yes)
+			)
+		)
+		(property "Datasheet" "~"
+			(at 107.95 69.85 0)
+			(effects
+				(font
+					(size 1.27 1.27)
+				)
+				(hide yes)
+			)
+		)
+		(property "Description" "test point"
+			(at 113.03 69.85 0)
+			(effects
+				(font
+					(size 1.27 1.27)
+				)
+				(hide yes)
+			)
+		)
+		(pin "1"
+		)
+		(instances
+			(project "Tracker"
+				(path "/60c5e70b-bc37-4402-aa86-9378cecb8f85/5d9555c7-4fd3-4187-a03c-c3d0cf6806ca"
+					(reference "T19")
 					(unit 1)
 				)
@@
 			)
 		)
-		(property "Footprint" "Package_SO:TSSOP-8_3x3mm_P0.65mm"
+		(property "Footprint" "Package_SO:SO-8_5.3x6.2mm_P1.27mm"
 			(at 96.52 78.74 0)
 			(effects
@@
 			)
 		)
-		(property "Footprint" "Crystal:Crystal_AT310_D3.0mm_L10.0mm_Horizontal"
+		(property "Footprint" "Crystal:Crystal_SMD_3215-2Pin_3.2x1.5mm"
 			(at 77.47 76.2 0)
 			(effects
@@
 		(fields_autoplaced yes)
 		(property "Reference" "R52"
-			(at 132.08 60.96 0)
+			(at 132.08 60.9599 0)
 			(effects
 				(font
@@
 			)
 		)
-		(property "Value" "270"
-			(at 132.08 63.5 0)
-			(effects
-				(font
+		(property "Value" "330"
+			(at 132.08 63.4999 0)
+			(effects
+				(font
