File: Hardware/V2_CMS/Modules/Reset.kicad_sch (KiCad schematic)
At the start: 3 parts, among them J11 USR_BTN, SW4 SW_B

Commit message: update of directory
Parts:
- J11: value USR_BTN -> RST_BUTTON
- SW4: footprint Button_Switch_THT:SW_PUSH_6mm_H8mm -> Button_Switch_SMD:SW_Push_1P1T_NO_CK_KSC7xxJ
Connections:
- net GND: now also J11.1 (Pin_1); no longer J11.2 (Pin_2)
- net RESET: now also J11.2 (Pin_2); no longer J11.1 (Pin_1)
Changed lines of the file:
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@@
 			)
 		)
-		(property "Footprint" "Button_Switch_THT:SW_PUSH_6mm_H8mm"
+		(property "Footprint" "Button_Switch_SMD:SW_Push_1P1T_NO_CK_KSC7xxJ"
 			(at 78.74 60.96 0)
 			(effects
@@
 	(symbol
 		(lib_id "Connector:Conn_01x02_Pin")
-		(at 60.96 58.42 0)
+		(at 60.96 60.96 0)
+		(mirror x)
 		(unit 1)
 		(exclude_from_sim no)
@@
 		(dnp no)
 		(property "Reference" "J11"
-			(at 59.69 60.9601 0)
+			(at 59.69 58.4199 0)
 			(effects
 				(font
@@
 			)
 		)
-		(property "Value" "USR_BTN"
-			(at 59.69 58.4201 0)
+		(property "Value" "RST_BUTTON"
+			(at 59.69 60.9599 0)
 			(effects
 				(font
@@
 		)
 		(property "Footprint" "TerminalBlock_Phoenix:TerminalBlock_Phoenix_MPT-0,5-2-2.54_1x02_P2.54mm_Horizontal"
-			(at 60.96 58.42 0)
+			(at 60.96 60.96 0)
 			(effects
 				(font
@@
 		)
 		(property "Datasheet" "~"
-			(at 60.96 58.42 0)
+			(at 60.96 60.96 0)
 			(effects
 				(font
@@
 		)
 		(property "Description" ""
-			(at 60.96 58.42 0)
+			(at 60.96 60.96 0)
 			(effects
 				(font
