File: Hardware/V2_CMS/Modules/Stepper.kicad_sch (KiCad schematic)
At the start: 2 parts, among them J15 PinHeader_Control, J16 Stepper

Commit message: update of directory
Parts:
- removed J15: PinHeader_Control, Connector_PinHeader_2.54mm:PinHeader_1x04_P2.54mm_Vertical, symbol Connector:Conn_01x04_Pin
- added C30: 100nF, Capacitor_SMD:C_0603_1608Metric, symbol Device:C
- added C31, C32: XX, Capacitor_SMD:C_0603_1608Metric, symbol Device:C
- added D22, D35: 1N4148, Diode_SMD:D_SOD-323, symbol Diode:1N4148
- added IC1: L6208, Package_SO:ST_PowerSSO-36_SlugDown_ThermalVias, symbol L6208:L6208
- added J22: Stepper_Pos, TerminalBlock_Phoenix:TerminalBlock_Phoenix_MPT-0,5-2-2.54_1x02_P2.54mm_Horizontal, symbol Connector:Screw_Terminal_01x02
- added J26: +24V, Connector_Phoenix_MSTB:PhoenixContact_MSTBA_2,5_2-G-5,08_1x02_P5.08mm_Horizontal, symbol Connector:Screw_Terminal_01x02
- added J31: Motor_Control_Pull_Up, TerminalBlock_Phoenix:TerminalBlock_Phoenix_MPT-0,5-3-2.54_1x03_P2.54mm_Horizontal, symbol Connector:Screw_Terminal_01x03
- added J32: Motor_Control, TerminalBlock_Phoenix:TerminalBlock_Phoenix_MPT-0,5-3-2.54_1x03_P2.54mm_Horizontal, symbol Connector:Screw_Terminal_01x03
- added R100, R101, R64, R97, R98, R99: 10k, Resistor_SMD:R_0603_1608Metric, symbol Device:R
- added R103: 0, Resistor_SMD:R_0603_1608Metric, symbol PCM_SL_Devices:Resistor_0.5W
- added R65, R66: XX, Resistor_SMD:R_0603_1608Metric, symbol Device:R
- added R79, R80: 0.33, Resistor_THT:R_Axial_DIN0414_L11.9mm_D4.5mm_P15.24mm_Horizontal, symbol Device:R
- added R84, R85, R86, R87, R88, R89: 220, Resistor_SMD:R_0603_1608Metric, symbol Device:R
- added RV2: Vref_B, Potentiometer_SMD:Potentiometer_Bourns_3314S_Horizontal, symbol Device:R_Potentiometer
- added RV3: Vref_A, Potentiometer_SMD:Potentiometer_Bourns_3314S_Horizontal, symbol Device:R_Potentiometer
- added T28, T29, T3, T30, T31, T32, T39, T42: TP, TestPoint:TestPoint_Pad_D1.0mm, symbol Connector:TestPoint
- added U23, U24, U25: PC817, Package_SO:SOP-4_4.4x2.6mm_P1.27mm, symbol Isolator:PC817
- J16: footprint TerminalBlock_Phoenix:TerminalBlock_Phoenix_MPT-0,5-4-2.54_1x04_P2.54mm_Horizontal -> Connector_Phoenix_MSTB:PhoenixContact_MSTBA_2,5_4-G-5,08_1x04_P5.08mm_Horizontal
Connections:
- net GND: now also C31.2, C32.2, IC1.18, IC1.19, IC1.23 (RESET), IC1.6, IC1.7, J22.1 (Pin_1), J26.1 (Pin_1), R100.2, R65.1, R66.1, R79.2, R80.2, R98.2, RV2.1, RV3.1, T39.1, U23.3, U24.3, U25.3; no longer J16.4 (Pin_4)
- net Dir: no longer names the net of J16.1 (Pin_1)
- net Dir: now also IC1.5 (OUT1A)
- net Enable: no longer names the net of J16.2 (Pin_2)
- net Enable: now also IC1.21 (OUT2A)
- net Pulse: no longer names the net of J16.3 (Pin_3)
- net Pulse: now also IC1.8 (OUT1B)
- new net: R103.1, R64.1
- new net: R85.1, U24.1
- new net: IC1.22 (VCP), R101.1
- new net: C30.2, R101.2
- new net: C30.1, D22.2 (A), D35.1 (K)
- new net: R84.1, U23.1
- new net: IC1.16 (OUT2B), J16.4 (Pin_4)
- new net: R86.1, U25.1
- new net: D22.1 (K), IC1.15 (VBOOT)
- new net +5V: J31.1 (Pin_1), J31.2 (Pin_2), J31.3 (Pin_3), R103.2, R84.2, R85.2, R86.2, R87.1, R88.1, R89.1, R97.1, R99.1, RV2.3, RV3.3
- new net CONTROL: IC1.13 (CONTROL), R97.2, R98.1, T42.1
- new net HALF/FULL: IC1.12 (HALF/FULL), R100.1, R99.2, T3.1
- new net RC_1: C31.1, IC1.4 (RCA), IC1.9 (RCB), R65.2, T28.1
- new net RC_2: C32.1, R66.2, T29.1
- new net SENSE_A: IC1.3 (SENSE_A), R80.1
- new net SENSE_B: IC1.10 (SENSE_B), R79.1
- new net STEP_CW: IC1.2 (CW/CWW), J32.1 (Pin_1), R88.2, T31.1, U24.4
- new net STEP_ENABLE: IC1.14 (EN), J32.2 (Pin_2), R87.2, T32.1, U25.4
- new net STEP_PULSE: IC1.1 (CLOCK), J32.3 (Pin_3), R89.2, T30.1, U23.4
- new net Stepper_CW/~{CCW}: U24.2
- new net Stepper_Enable: U25.2
- new net Stepper_Pulse: U23.2
- new net Vcc: D35.2 (A), IC1.17 (VS_B), IC1.20 (VS_A), J26.2 (Pin_2)
- new net Vref_A: IC1.24 (VREF_A), RV3.2
- new net Vref_B: IC1.11 (VREF_B), RV2.2
- new net ~{Stepper_Origine}: J22.2 (Pin_2), R64.2
Other:
- title: Stepper connector -> Stepper controller
- moved on the sheet: J16
