File: Hardware/V2_CMS/Modules/WIND.kicad_sch (KiCad schematic)
At the start: 18 parts, among them J1 Wind, J2 RAW_data_Wind, U1 LM358, U2 74HC123

Commit message: update of directory
Parts:
- removed J2: RAW_data_Wind, Connector_PinHeader_2.54mm:PinHeader_1x01_P2.54mm_Vertical, symbol Connector:Conn_01x01_Pin
- removed JP1: Jumper, Connector_PinHeader_2.54mm:PinHeader_1x02_P2.54mm_Vertical, symbol Jumper:Jumper_2_Bridged
- removed RV1: R_Potentiometer, Potentiometer_THT:Potentiometer_Bourns_3266Y_Vertical, symbol Device:R_Potentiometer
- added C27: 100nF, Capacitor_SMD:C_0603_1608Metric, symbol Device:C
- added J2, J20: 132415, Connector_Coaxial:SMA_Molex_73251-1153_EdgeMount_Horizontal, symbol Connector:Conn_Coaxial
- added R104, R105: 0, Resistor_SMD:R_0603_1608Metric, symbol PCM_SL_Devices:Resistor_0.5W
- added R60: 0, Resistor_SMD:R_0603_1608Metric, symbol Device:R
- added T10, T11, T12, T41, T9: TP, TestPoint:TestPoint_Pad_D1.0mm, symbol Connector:TestPoint
- added U22: MCP4011, Package_SO:SOIC-8_3.9x4.9mm_P1.27mm, symbol Potentiometer_Digital:MCP4011-xxxxSN
- R10: value 270 -> 330
- U1: value LM358 -> LM358DR; footprint Package_SO:TSSOP-8_3x3mm_P0.65mm -> Package_SO:TSSOP-8_4.4x3mm_P0.65mm
- U2: value 74HC123 -> 74HC123D; footprint Package_SO:SSOP-16_4.4x5.2mm_P0.65mm -> Package_SO:SOIC-16W_5.3x10.2mm_P1.27mm
Connections:
- net +5V: now also C27.2, U22.1 (VDD), U22.3 (A)
- net GND: now also C27.1, J2.2 (Ext), J20.2 (Ext), U22.2 (VSS), U22.6 (B)
- net at D1.2 (A): now also R60.1
- net Simulation: now reaches U2.1 (A)
- net Simulation: now also T41.1
- net at R6.1, U2.13 (Q): now also T9.1
- net at J1.1 (Pin_1), R4.2, U2.2 (B): now also J2.1 (In)
- net at C4.1, R6.2, U1.5 (+): now also J20.1 (In)
- net at U1.2 (-): now also T12.1, U22.4 (W)
- net at R7.1, U1.6 (-), U1.7: now also T10.1
- net Wind_interrupt: no longer names the net of R8.2, R9.2, U1.1
- net Wind_interrupt: now also R104.1, R105.1, R60.2, T11.1
- new net U/~{D}: U22.8 (U/~{D})
- new net Wind_interrupt_MCU: R105.2
- new net Wind_interrupt_Power: R104.2
- new net ~{CS}: U22.5 (~{CS})
- no-connect marks 9 -> 8
