File: Hardware/V2_CMS/Modules/Wifi.kicad_sch (KiCad schematic)
At the start: 2 parts, among them U14 NRF24L01_Breakout

Commit message: update of directory
Parts:
- added C28: 4.7u, Capacitor_SMD:C_0603_1608Metric, symbol Device:C
Connections:
- net +3.3V: now also C28.1
- net ESP_GND: now also C28.2
Changed lines of the file:
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@@
+	)
+	(junction
+		(at 110.49 27.94)
+		(diameter 0)
+		(color 0 0 0 0)
 	)
 	(junction
@@
 	(wire
 		(pts
-			(xy 110.49 31.75) (xy 110.49 35.56)
+			(xy 110.49 25.4) (xy 110.49 27.94)
 		)
 		(stroke
@@
 		)
 	)
+	(wire
+		(pts
+			(xy 106.68 27.94) (xy 110.49 27.94)
+		)
+		(stroke
+			(width 0)
+			(type default)
+		)
+	)
 	(bus
 		(pts
@@
 	(wire
 		(pts
-			(xy 111.76 31.75) (xy 110.49 31.75)
+			(xy 111.76 25.4) (xy 110.49 25.4)
 		)
 		(stroke
@@
 		(pts
 			(xy 66.04 35.56) (xy 57.15 35.56)
+		)
+		(stroke
+			(width 0)
+			(type default)
+		)
+	)
+	(wire
+		(pts
+			(xy 96.52 27.94) (xy 99.06 27.94)
+		)
+		(stroke
+			(width 0)
+			(type default)
+		)
+	)
+	(wire
+		(pts
+			(xy 110.49 27.94) (xy 110.49 35.56)
 		)
 		(stroke
@@
 		)
 	)
+	(label "GND"
+		(at 96.52 27.94 180)
+		(fields_autoplaced yes)
+		(effects
+			(font
+				(size 1.27 1.27)
+			)
+			(justify right bottom)
+		)
+	)
 	(label "MOSI"
 		(at 66.04 38.1 180)
@@
 	(hierarchical_label "+3.3V"
 		(shape input)
-		(at 111.76 31.75 0)
+		(at 111.76 25.4 0)
 		(fields_autoplaced yes)
 		(effects
@@
 	)
 	(hierarchical_label "ESP_CE"
-		(shape bidirectional)
+		(shape input)
 		(at 93.98 62.23 180)
 		(fields_autoplaced yes)
@@
 			)
 			(justify right)
+		)
+	)
+	(symbol
+		(lib_id "Device:C")
+		(at 102.87 27.94 270)
+		(unit 1)
+		(exclude_from_sim no)
+		(in_bom yes)
+		(on_board yes)
+		(dnp no)
+		(property "Reference" "C28"
+			(at 104.902 29.972 90)
+			(effects
+				(font
+					(size 1.27 1.27)
+				)
+				(justify left)
+			)
+		)
+		(property "Value" "4.7u"
+			(at 94.996 30.226 90)
+			(effects
+				(font
+					(size 1.27 1.27)
+				)
+				(justify left)
+			)
+		)
+		(property "Footprint" "Capacitor_SMD:C_0603_1608Metric"
+			(at 99.06 28.9052 0)
+			(effects
+				(font
+					(size 1.27 1.27)
+				)
+				(hide yes)
+			)
+		)
+		(property "Datasheet" "~"
+			(at 102.87 27.94 0)
+			(effects
+				(font
+					(size 1.27 1.27)
+				)
+				(hide yes)
+			)
+		)
+		(property "Description" ""
+			(at 102.87 27.94 0)
+			(effects
+				(font
+					(size 1.27 1.27)
+				)
+				(hide yes)
+			)
+		)
+		(pin "1"
+		)
+		(pin "2"
+		)
+		(instances
+			(project "Tracker"
+				(path "/60c5e70b-bc37-4402-aa86-9378cecb8f85/67c447e5-4ef9-49b2-8c11-c6a3219ed198"
+					(reference "C28")
+					(unit 1)
+				)
+			)
 		)
 	)
@@
 		(dnp no)
 		(property "Reference" "C21"
-			(at 105.41 36.83 0)
+			(at 104.902 37.592 90)
 			(effects
 				(font
@@
 		)
 		(property "Value" "100nF"
-			(at 100.076 36.322 0)
-			(effects
-				(font
+			(at 94.996 37.846 90)
+			(effects
+				(font
