File: Hardware/V2_CMS/Modules/Xtal.kicad_sch (KiCad schematic)
At the start: 3 parts, among them Y1 16MHz

Commit message: update of directory
Parts:
- Y1: footprint Crystal:Crystal_HC49-4H_Vertical -> Crystal:Crystal_SMD_HC49-SD
Changed lines of the file:
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@@
 			)
 		)
-		(property "Footprint" "Crystal:Crystal_HC49-4H_Vertical"
+		(property "Footprint" "Crystal:Crystal_SMD_HC49-SD"
 			(at 95.25 55.88 0)
 			(effects
