File: Hardware/V2_CMS_4_Layers/Modules/GNSS.kicad_sch (KiCad schematic)
At the start: 57 parts, among them J10 132415, J5 USB_C_Receptacle_USB2.0_16P, Q1 SI2302, Q10 CJ3401, Q11 2N7002, T1 TP, T33 TP, T34 TP, T38 TP, T4 TP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

Commit message: Update 4Layers
Other:
- note added: "MUST BE REPLACED By BSS"
Changed lines of the file:
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@@
+		)
+	)
+	(text "MUST BE REPLACED By BSS"
+		(exclude_from_sim no)
+		(at 200.406 155.702 0)
+		(effects
+			(font
+				(size 1.27 1.27)
+			)
 		)
 	)
